File: prj/nuku-carrier-template-bare/core-east.kicad_sch (KiCad schematic)
At the start: 1 part, among them J2 DF40HC(4.0)-90DS-0.4V

Commit message: Update nuku.carrier.template to template.bare
Other:
- company: (none) -> Samuel López Asunción
- title: (none) -> nuku.carrier.template.bare / core-east-34
Changed lines of the file:
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@@
 	(generator_version "9.0")
 	(paper "A4")
+	(title_block
+		(title "nuku.carrier.template.bare / core-east-34")
+		(date "2025-06-09")
+		(rev "0")
+		(company "Samuel López Asunción")
+		(comment 1 "@supersmau")
+	)
 	(junction
 		(at 158.75 53.34)
