File: prj/nuku-carrier-template-bare/core-south.kicad_sch (KiCad schematic)
At the start: 19 parts, among them J1 DF40HC(4.0)-90DS-0.4V, SW1 PROG

Commit message: Update nuku.carrier.template to template.bare
Other:
- company: (none) -> Samuel López Asunción
- title: (none) -> nuku.carrier.template.bare / core-south-0
Changed lines of the file:
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@@
 	(generator_version "9.0")
 	(paper "A4")
+	(title_block
+		(title "nuku.carrier.template.bare / core-south-0")
+		(date "2025-06-09")
+		(rev "0")
+		(company "Samuel López Asunción")
+		(comment 1 "@supersmau")
+	)
 	(rectangle
 		(start 24.13 22.86)

Commit message: Route template.basic
Other:
- moved on the sheet: R1, R10, R11, R2, R3, R4, R5, R6, R9
Changed lines of the file:
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@@
 	(symbol
 		(lib_id "Device:R")
-		(at 64.77 104.14 0)
-		(mirror x)
+		(at 64.77 104.14 180)
 		(unit 1)
 		(exclude_from_sim no)
@@
 		(dnp no)
 		(property "Reference" "R4"
-			(at 66.04 111.76 90)
+			(at 63.5 111.76 90)
 			(effects
 				(font
@@
 		)
 		(property "Value" "1k"
-			(at 66.04 100.33 90)
+			(at 63.5 100.33 90)
 			(effects
 				(font
@@
 		)
 		(property "Footprint" "Resistor_SMD:R_0402_1005Metric"
-			(at 62.992 104.14 90)
+			(at 66.548 104.14 90)
 			(effects
 				(font
@@
 	(symbol
 		(lib_id "Device:R")
-		(at 57.15 144.78 0)
-		(mirror x)
+		(at 57.15 144.78 180)
 		(unit 1)
 		(exclude_from_sim no)
@@
 		(dnp no)
 		(property "Reference" "R11"
-			(at 58.42 152.4 90)
+			(at 55.88 152.4 90)
 			(effects
 				(font
@@
 		)
 		(property "Value" "4k7"
-			(at 58.42 140.97 90)
+			(at 55.88 140.97 90)
 			(effects
 				(font
@@
 		)
 		(property "Footprint" "Resistor_SMD:R_0402_1005Metric"
-			(at 55.372 144.78 90)
+			(at 58.928 144.78 90)
 			(effects
 				(font
@@
 	(symbol
 		(lib_id "Device:R")
-		(at 52.07 144.78 0)
-		(mirror x)
+		(at 52.07 144.78 180)
 		(unit 1)
 		(exclude_from_sim no)
@@
 		(dnp no)
 		(property "Reference" "R9"
-			(at 53.34 152.4 90)
+			(at 50.8 152.4 90)
 			(effects
 				(font
@@
 		)
 		(property "Value" "330"
-			(at 53.34 140.97 90)
+			(at 50.8 140.97 90)
 			(effects
 				(font
@@
 		)
 		(property "Footprint" "Resistor_SMD:R_0402_1005Metric"
-			(at 50.292 144.78 90)
+			(at 53.848 144.78 90)
 			(effects
 				(font
@@
 	(symbol
 		(lib_id "Device:R")
-		(at 69.85 81.28 0)
-		(mirror x)
+		(at 69.85 81.28 180)
 		(unit 1)
 		(exclude_from_sim no)
@@
 		(dnp no)
 		(property "Reference" "R3"
-			(at 71.12 88.9 90)
+			(at 68.58 88.9 90)
 			(effects
 				(font
@@
 		)
 		(property "Value" "1k"
-			(at 71.12 77.47 90)
+			(at 68.58 77.47 90)
 			(effects
 				(font
@@
 		)
 		(property "Footprint" "Resistor_SMD:R_0402_1005Metric"
-			(at 68.072 81.28 90)
+			(at 71.628 81.28 90)
 			(effects
 				(font
@@
 	(symbol
 		(lib_id "Device:R")
-		(at 64.77 81.28 0)
-		(mirror x)
+		(at 64.77 81.28 180)
 		(unit 1)
 		(exclude_from_sim no)
@@
 		(dnp yes)
 		(property "Reference" "R1"
-			(at 66.04 88.9 90)
+			(at 63.5 88.9 90)
 			(effects
 				(font
@@
 		)
 		(property "Value" "1k"
-			(at 66.04 77.47 90)
+			(at 63.5 77.47 90)
 			(effects
 				(font
@@
 		)
 		(property "Footprint" "Resistor_SMD:R_0402_1005Metric"
-			(at 62.992 81.28 90)
+			(at 66.548 81.28 90)
 			(effects
 				(font
@@
 	(symbol
 		(lib_id "Device:R")
-		(at 54.61 144.78 0)
-		(mirror x)
+		(at 54.61 144.78 180)
 		(unit 1)
 		(exclude_from_sim no)
@@
 		(dnp no)
 		(property "Reference" "R10"
-			(at 55.88 152.4 90)
+			(at 53.34 152.4 90)
 			(effects
 				(font
@@
 		)
 		(property "Value" "4k7"
-			(at 55.88 140.97 90)
+			(at 53.34 140.97 90)
 			(effects
 				(font
@@
 		)
 		(property "Footprint" "Resistor_SMD:R_0402_1005Metric"
-			(at 52.832 144.78 90)
+			(at 56.388 144.78 90)
 			(effects
 				(font
@@
 	(symbol
 		(lib_id "Device:R")
-		(at 67.31 104.14 0)
-		(mirror x)
+		(at 67.31 104.14 180)
 		(unit 1)
 		(exclude_from_sim no)
@@
 		(dnp no)
 		(property "Reference" "R5"
-			(at 68.58 111.76 90)
+			(at 66.04 111.76 90)
 			(effects
 				(font
@@
 		)
 		(property "Value" "1k"
-			(at 68.58 100.33 90)
+			(at 66.04 100.33 90)
 			(effects
 				(font
@@
 		)
 		(property "Footprint" "Resistor_SMD:R_0402_1005Metric"
-			(at 65.532 104.14 90)
+			(at 69.088 104.14 90)
 			(effects
 				(font
@@
 	(symbol
 		(lib_id "Device:R")
-		(at 67.31 81.28 0)
-		(mirror x)
+		(at 67.31 81.28 180)
 		(unit 1)
 		(exclude_from_sim no)
@@
 		(dnp yes)
 		(property "Reference" "R2"
-			(at 68.58 88.9 90)
+			(at 66.04 88.9 90)
 			(effects
 				(font
@@
 		)
 		(property "Value" "1k"
-			(at 68.58 77.47 90)
+			(at 66.04 77.47 90)
 			(effects
 				(font
@@
 		)
 		(property "Footprint" "Resistor_SMD:R_0402_1005Metric"
-			(at 65.532 81.28 90)
+			(at 69.088 81.28 90)
 			(effects
 				(font
@@
 	(symbol
 		(lib_id "Device:R")
-		(at 69.85 104.14 0)
-		(mirror x)
+		(at 69.85 104.14 180)
 		(unit 1)
 		(exclude_from_sim no)
@@
 		(dnp yes)
 		(property "Reference" "R6"
-			(at 71.12 111.76 90)
+			(at 68.58 111.76 90)
 			(effects
 				(font
@@
 		)
 		(property "Value" "1k"
-			(at 71.12 100.33 90)
+			(at 68.58 100.33 90)
 			(effects
 				(font
@@
 		)
 		(property "Footprint" "Resistor_SMD:R_0402_1005Metric"
-			(at 68.072 104.14 90)
-			(effects
-				(font
+			(at 71.628 104.14 90)
+			(effects
+				(font

Commit message: Finish template.basic + Production outputs
Connections:
- net MGTP_CLK0_P: no longer J1.32
- new net MGTP_CLK0_N: J1.32
Changed lines of the file:
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@@
 		)
 	)
-	(label "MGTP_CLK0_P"
+	(label "MGTP_CLK0_N"
 		(at 191.77 119.38 0)
 		(effects
