File: prj/nuku-carrier-template-bare/nuku-carrier-template-bare.kicad_pcb (KiCad board)
At the start: 4 copper layers, 48 x 65 mm, 24 parts, among them J1 DF40HC(4.0)-90DS-0.4V, J2 DF40HC(4.0)-90DS-0.4V, J3 DF40HC(4.0)-90DS-0.4V, J4 DF40HC(4.0)-90DS-0.4V, SW1 PROG

Commit message: Update nuku.carrier.template to template.bare
Other:
- board text added: "carrier.template.bare"
- board text removed: "carrier.template"
Changed lines of the file:
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@@
 	)
 	(paper "A4")
+	(title_block
+		(title "nuku.carrier.template.base")
+		(date "2025-06-09")
+		(rev "0")
+		(company "Samuel López Asunción")
+		(comment 1 "@supersmau")
+	)
 	(layers
 		(0 "F.Cu" signal "L1_(Sig).Cu")
 		(4 "In1.Cu" power "L2_(GND).Cu")
-		(6 "In2.Cu" power "L3_(PWR).Cu")
+		(6 "In2.Cu" power "L3_(GND).Cu")
 		(2 "B.Cu" signal "L4_(Sig).Cu")
 		(9 "F.Adhes" user "F.Adhesive")
@@
 		(layer "Edge.Cuts")
 	)
-	(gr_text "carrier.template"
+	(gr_text "carrier.template.bare"
 		(at 129.1 142 0)
 		(layer "F.SilkS")
@@
 			(justify left bottom)
 		)
-		(render_cache "carrier.template" 0
+		(render_cache "carrier.template.bare" 0
 			(polygon
 				(pts
@@
 				)
 			)
+			(polygon
+				(pts
+					(xy 144.091503 141.762) (xy 144.039389 141.756106) (xy 143.996726 141.739428) (xy 143.961395 141.712247)
+					(xy 143.934215 141.676656) (xy 143.918149 141.637238) (xy 143.912669 141.592654) (xy 143.91843 141.543121)
+					(xy 143.934739 141.502694) (xy 143.961395 141.469299) (xy 143.996439 141.444369) (xy 144.039104 141.428896)
+					(xy 144.091503 141.423393) (xy 144.143268 141.428876) (xy 144.185614 141.444331) (xy 144.220586 141.469299)
+					(xy 144.247293 141.5027) (xy 144.263628 141.543128) (xy 144.269398 141.592654) (xy 144.263909 141.637233)
+					(xy 144.247817 141.676649) (xy 144.220586 141.712247) (xy 144.185327 141.73947) (xy 144.142984 141.756127)
+				)
+			)
+			(polygon
+				(pts
+					(xy 144.948747 140.948268) (xy 145.004218 140.894078) (xy 145.070648 140.848849) (xy 145.119713 140.827162)
+					(xy 145.177037 140.813502) (xy 145.244269 140.808671) (xy 145.315395 140.815911) (xy 145.37723 140.836797)
+					(xy 145.431737 140.87116) (xy 145.476649 140.917387) (xy 145.512289 140.977261) (xy 145.538337 141.053671)
+					(xy 145.550106 141.134038) (xy 145.548361 141.231132) (xy 145.530216 141.348509) (xy 145.500473 141.456212)
+					(xy 145.462562 141.544164) (xy 145.417385 141.615366) (xy 145.36523 141.67224) (xy 145.302579 141.719706)
+					(xy 145.236114 141.752966) (xy 145.164857 141.772972) (xy 145.087489 141.77978) (xy 144.9952 141.770168)
+					(xy 144.919169 141.743022) (xy 144.85454 141.698084) (xy 144.803422 141.636337) (xy 144.766151 141.762)
+					(xy 144.486871 141.762) (xy 144.560638 141.415187) (xy 144.852149 141.415187) (xy 144.878498 141.469501)
+					(xy 144.92293 141.517427) (xy 144.959942 141.54156) (xy 145.000075 141.555896) (xy 145.044405 141.560768)
+					(xy 145.089199 141.55385) (xy 145.129301 141.533128) (xy 145.166306 141.496654) (xy 145.194951 141.451436)
+					(xy 145.220938 141.389363) (xy 145.243328 141.306279) (xy 145.25718 141.210729) (xy 145.254448 141.143173)
+					(xy 145.239994 141.096157) (xy 145.212184 141.057895) (xy 145.175674 141.035554) (xy 145.127581 141.027683)
+					(xy 145.077605 141.033405) (xy 145.031924 141.050337) (xy 144.9904 141.076067) (xy 144.954047 141.107697)
+					(xy 144.922632 141.143446) (xy 144.898054 141.178992) (xy 144.852149 141.415187) (xy 144.560638 141.415187)
+					(xy 144.760338 140.476305) (xy 145.050132 140.476305)
+				)
+			)
+			(polygon
+				(pts
+					(xy 146.338111 140.814104) (xy 146.419003 140.829786) (xy 146.49292 140.857908) (xy 146.552873 140.898003)
+					(xy 146.585272 140.932218) (xy 146.610398 140.97342) (xy 146.628356 141.022811) (xy 146.636788 141.07491)
+					(xy 146.636028 141.13809) (xy 146.624082 141.21481) (xy 146.50748 141.762) (xy 146.241536 141.762)
+					(xy 146.254958 141.649758) (xy 146.189622 141.706858) (xy 146.122456 141.746783) (xy 146.04679 141.770849)
+					(xy 145.9461 141.77978) (xy 145.856594 141.77026) (xy 145.782995 141.743364) (xy 145.740793 141.714991)
+					(xy 145.707266 141.679159) (xy 145.68161 141.634969) (xy 145.666325 141.585994) (xy 145.661171 141.527893)
+					(xy 145.663501 141.503311) (xy 145.952003 141.503311) (xy 145.959451 141.531303) (xy 145.975165 141.553416)
+					(xy 146.010489 141.575834) (xy 146.057915 141.583763) (xy 146.109829 141.577851) (xy 146.157419 141.56034)
+					(xy 146.200856 141.534527) (xy 146.237262 141.505374) (xy 146.287442 141.450834) (xy 146.315225 141.337908)
+					(xy 146.141879 141.34608) (xy 146.0474 141.364922) (xy 145.99957 141.389241) (xy 145.96939 141.422728)
+					(xy 145.953709 141.467076) (xy 145.952003 141.503311) (xy 145.663501 141.503311) (xy 145.667761 141.458357)
+					(xy 145.684295 141.398034) (xy 145.708779 141.349287) (xy 145.740851 141.310126) (xy 145.80357 141.263804)
+					(xy 145.886261 141.229599) (xy 145.979534 141.208176) (xy 146.093306 141.19455) (xy 146.349675 141.182069)
+					(xy 146.355403 141.144285) (xy 146.358194 141.096598) (xy 146.350102 141.062903) (xy 146.332057 141.035988)
+					(xy 146.30565 141.01734) (xy 146.273176 141.006642) (xy 146.232988 141.002807) (xy 146.172234 141.01044)
+					(xy 146.117669 141.032983) (xy 146.087889 141.056858) (xy 146.066475 141.089263) (xy 146.053213 141.132317)
+					(xy 145.782482 141.132317) (xy 145.802242 141.049644) (xy 145.83377 140.982594) (xy 145.876514 140.928389)
+					(xy 145.931226 140.885265) (xy 146.017075 140.844276) (xy 146.121393 140.818078) (xy 146.24829 140.808671)
+				)
+			)
+			(polygon
+				(pts
+					(xy 146.758293 141.762) (xy 146.956277 140.826452) (xy 147.237437 140.826452) (xy 147.205893 140.983744)
+					(xy 147.245173 140.928406) (xy 147.28766 140.885052) (xy 147.333522 140.852183) (xy 147.384567 140.828464)
+					(xy 147.442298 140.813786) (xy 147.508082 140.808671) (xy 147.543473 140.808671) (xy 147.493721 141.048713)
+					(xy 147.46987 141.048713) (xy 147.364638 141.055466) (xy 147.31319 141.065974) (xy 147.264193 141.083933)
+					(xy 147.219128 141.110639) (xy 147.17717 141.149072) (xy 147.047147 141.762)
+				)
+			)
+			(polygon
+				(pts
+					(xy 148.171438 140.816766) (xy 148.25439 140.839737) (xy 148.32549 140.876546) (xy 148.386641 140.927615)
+					(xy 148.434191 140.990541) (xy 148.468934 141.067177) (xy 148.487596 141.149817) (xy 148.490879 141.244641)
+					(xy 148.476627 141.354407) (xy 147.824377 141.354407) (xy 147.822512 141.410503) (xy 147.830104 141.461862)
+					(xy 147.849223 141.507607) (xy 147.881224 141.543243) (xy 147.925612 141.565687) (xy 147.991756 141.574189)
+					(xy 148.059379 141.566196) (xy 148.111777 141.544013) (xy 148.139901 141.520679) (xy 148.161361 141.489759)
+					(xy 148.176318 141.449637) (xy 148.462266 141.449637) (xy 148.432574 141.533544) (xy 148.39448 141.601943)
+					(xy 148.348382 141.657172) (xy 148.293946 141.700878) (xy 148.232335 141.733641) (xy 148.15932 141.758321)
+					(xy 148.072895 141.774137) (xy 147.970727 141.77978) (xy 147.871649 141.772184) (xy 147.78807 141.750764)
+					(xy 147.717264 141.716778) (xy 147.655705 141.668856) (xy 147.607402 141.609402) (xy 147.571427 141.536747)
+					(xy 147.55065 141.457641) (xy 147.543755 141.365407) (xy 147.552791 141.257211) (xy 147.57093 141.176513)
+					(xy 147.857801 141.176513) (xy 148.21453 141.176513) (xy 148.214803 141.122783) (xy 148.203075 141.082308)
+					(xy 148.180322 141.049295) (xy 148.148536 141.025717) (xy 148.11014 141.011603) (xy 148.064419 141.006654)
+					(xy 148.011815 141.011893) (xy 147.967259 141.026829) (xy 147.929096 141.051106) (xy 147.89785 141.083833)
+					(xy 147.874053 141.125048) (xy 147.857801 141.176513) (xy 147.57093 141.176513) (xy 147.573965 141.163013)
+					(xy 147.6046 141.082126) (xy 147.644089 141.012724) (xy 147.694341 140.951125) (xy 147.753016 140.900698)
+					(xy 147.820957 140.860646) (xy 147.895027 140.832437) (xy 147.978812 140.814826) (xy 148.073993 140.808671)
+				)
+			)
