File: prj/nuku-carrier-template-basic/nuku-carrier-template-basic.kicad_pcb (KiCad board)
At the start: 4 copper layers, 48 x 65 mm, 24 parts, among them J1 DF40HC(4.0)-90DS-0.4V, J2 DF40HC(4.0)-90DS-0.4V, J3 DF40HC(4.0)-90DS-0.4V, J4 DF40HC(4.0)-90DS-0.4V, SW1 PROG

Commit message: Route template.basic
Parts:
- removed R13, R14: 10k, Resistor_SMD:R_0402_1005Metric
- removed the R8 at (144.1, 117.0)
- added ?: MountingHole_3.2mm_M3_Pad_TopBottom, MountingHole:MountingHole_3.2mm_M3_Pad_TopBottom, F.Cu at (96.5, 131.0)
- added ?: MountingHole_3.2mm_M3_Pad_TopBottom, MountingHole:MountingHole_3.2mm_M3_Pad_TopBottom, F.Cu at (188.5, 79.0)
- added ?: MountingHole_3.2mm_M3_Pad_TopBottom, MountingHole:MountingHole_3.2mm_M3_Pad_TopBottom, F.Cu at (96.5, 79.0)
- added ?: MountingHole_3.2mm_M3_Pad_TopBottom, MountingHole:MountingHole_3.2mm_M3_Pad_TopBottom, F.Cu at (188.5, 131.0)
- added C1: 4u7, Capacitor_SMD:C_0603_1608Metric, F.Cu at (105.7, 121.4)
- added C10: 33p, Capacitor_SMD:C_0402_1005Metric, F.Cu at (110.1, 95.2)
- added C11: 470n, Capacitor_SMD:C_0402_1005Metric, F.Cu at (110.7, 106.8)
- added C12: 470n, Capacitor_SMD:C_0402_1005Metric, F.Cu at (110.7, 103.0)
- added C13: 4u7, Capacitor_SMD:C_0603_1608Metric, F.Cu at (123.9, 101.2)
- added C14: 33p, Capacitor_SMD:C_0402_1005Metric, F.Cu at (106.5, 98.2)
- added C15: 470n, Capacitor_SMD:C_0402_1005Metric, F.Cu at (110.7, 108.8)
- added C16: 470n, Capacitor_SMD:C_0402_1005Metric, F.Cu at (123.9, 108.2)
- added C17: 470n, Capacitor_SMD:C_0402_1005Metric, F.Cu at (116.1, 112.0)
- added C18: 470n, Capacitor_SMD:C_0402_1005Metric, F.Cu at (113.5, 98.8)
- added C19: 470n, Capacitor_SMD:C_0402_1005Metric, F.Cu at (121.1, 112.0)
- added C2: 33p, Capacitor_SMD:C_0402_1005Metric, F.Cu at (108.7, 118.8)
- added C20: 470n, Capacitor_SMD:C_0402_1005Metric, F.Cu at (123.9, 103.8)
- added C21: 470n, Capacitor_SMD:C_0402_1005Metric, F.Cu at (117.7, 98.8)
- added C22: 470n, Capacitor_SMD:C_0402_1005Metric, F.Cu at (115.7, 82.4)
- added C23: 470n, Capacitor_SMD:C_0402_1005Metric, F.Cu at (120.1, 81.8)
- added C3: 47u, Capacitor_SMD:C_0805_2012Metric, F.Cu at (110.5, 121.4)
- added C4: 470n, Capacitor_SMD:C_0402_1005Metric, F.Cu at (98.7, 98.2)
- added C5: 47u, Capacitor_SMD:C_0805_2012Metric, F.Cu at (99.3, 112.0)
- added C6: 470n, Capacitor_SMD:C_0402_1005Metric, F.Cu at (112.7, 90.2)
- added C7: 4u7, Capacitor_SMD:C_0603_1608Metric, F.Cu at (109.3, 107.2)
- added C8: 4u7, Capacitor_SMD:C_0603_1608Metric, F.Cu at (109.3, 103.0)
- added C9: 4u7, Capacitor_SMD:C_0603_1608Metric, F.Cu at (120.5, 99.2)
- added D2: PWR, LED_SMD:LED_0805_2012Metric, F.Cu at (97.1, 117.0)
- added D3: RX, LED_SMD:LED_0805_2012Metric, F.Cu at (97.1, 88.0)
- added D4: TX, LED_SMD:LED_0805_2012Metric, F.Cu at (97.1, 93.0)
- added J5: USB_C_Receptacle_USB2.0_16P, nuku:TYPE-C16PIN, F.Cu at (92.5, 105.0)
- added J6: TC2050, Connector:Tag-Connect_TC2050-IDC-NL_2x05_P1.27mm_Vertical, F.Cu at (121.1, 121.4)
- added J7: PMOD_A, nuku:PMOD_PinSocket_2x06_P2.54mm_Horizontal, F.Cu at (192.5, 93.6)
- added J8: PMOD_B, nuku:PMOD_PinSocket_2x06_P2.54mm_Horizontal, F.Cu at (192.5, 116.4)
- added L1: 1u, Inductor_SMD:L_Changjiang_FNR252010S, F.Cu at (107.7, 124.4)
- added L2: 600, Inductor_SMD:L_0603_1608Metric, F.Cu at (107.7, 107.2)
- added L3: 600, Inductor_SMD:L_0603_1608Metric, F.Cu at (107.7, 103.0)
- added R19: 100k, Resistor_SMD:R_0402_1005Metric, F.Cu at (103.7, 120.8)
- added R20: 200k, Resistor_SMD:R_0402_1005Metric, F.Cu at (103.7, 122.0)
- added R21: 100k, Resistor_SMD:R_0402_1005Metric, F.Cu at (106.7, 117.6)
- added R22: 22k, Resistor_SMD:R_0402_1005Metric, F.Cu at (108.7, 117.6)
- added R23: 1k, Resistor_SMD:R_0402_1005Metric, F.Cu at (97.1, 119.4)
- added R24: 1M, Resistor_SMD:R_0402_1005Metric, F.Cu at (99.9, 98.2)
- added R25: 5k1, Resistor_SMD:R_0402_1005Metric, F.Cu at (103.9, 102.6)
- added R26: 5k1, Resistor_SMD:R_0402_1005Metric, F.Cu at (103.9, 107.4)
- added R30: 10k, Resistor_SMD:R_0402_1005Metric, F.Cu at (118.3, 94.4)
- added R31: 10k, Resistor_SMD:R_0402_1005Metric, F.Cu at (118.3, 93.2)
- added R32: 10k, Resistor_SMD:R_0402_1005Metric, F.Cu at (118.3, 92.0)
- added R33: 2k2, Resistor_SMD:R_0402_1005Metric, F.Cu at (115.9, 99.2)
- added R34: 12k, Resistor_SMD:R_0402_1005Metric, F.Cu at (107.7, 112.0)
- added R35: 1k, Resistor_SMD:R_0402_1005Metric, F.Cu at (109.3, 112.0)
- added R36: 1k, Resistor_SMD:R_0402_1005Metric, F.Cu at (97.1, 85.6)
- added R37: 1k, Resistor_SMD:R_0402_1005Metric, F.Cu at (97.1, 90.6)
- added R38: 0, Resistor_SMD:R_0402_1005Metric, F.Cu at (121.1, 115.4)
- added R41: 4k7, Resistor_SMD:R_0402_1005Metric, F.Cu at (103.9, 83.0)
- added R42: 4k7, Resistor_SMD:R_0402_1005Metric, F.Cu at (83.0, 67.7)
- added R43: 4k7, Resistor_SMD:R_0402_1005Metric, F.Cu at (83.0, 69.7)
- added SW2: RESET, nuku:TS-1088-AR02016, F.Cu at (78.3, 69.0)
- added U1: AP61302, Package_TO_SOT_SMD:SOT-563, F.Cu at (107.7, 121.4)
- added U10: SRV05-4, Package_TO_SOT_SMD:SOT-23-6, F.Cu at (173.5, 119.4)
- added U2: SRV05-4, Package_TO_SOT_SMD:SOT-23-6, F.Cu at (103.9, 105.0)
- added U3: M93C56-WDW6TP, Package_SO:TSSOP-8_4.4x3mm_P0.65mm, F.Cu at (115.1, 93.2)
- added U4: FT2232HQ, Package_DFN_QFN:QFN-64-1EP_9x9mm_P0.5mm_EP4.35x4.35mm, F.Cu at (117.5, 105.6)
- added U5: IS25LP064A, Package_SO:SOIC-8_5.3x5.3mm_P1.27mm, F.Cu at (109.5, 84.4)
- added U6: OT3225100MJBA4SL, Crystal:Crystal_SMD_3225-4Pin_3.2x2.5mm, F.Cu at (120.7, 84.4)
- added U7: SRV05-4, Package_TO_SOT_SMD:SOT-23-6, F.Cu at (173.5, 90.6)
- added U8: SRV05-4, Package_TO_SOT_SMD:SOT-23-6, F.Cu at (173.5, 113.4)
- added U9: SRV05-4, Package_TO_SOT_SMD:SOT-23-6, F.Cu at (173.5, 96.6)
- added Y1: 12 MHz, Crystal:Crystal_SMD_3225-4Pin_3.2x2.5mm, F.Cu at (109.3, 97.6)
- R12: value 330 -> 1k
- moved SW1 61.5 mm to (80.9, 123.8)
- moved D1 53.3 mm to (97.1, 122.0), turned to 90 degrees
- moved R12 50.3 mm to (97.1, 124.4), turned to 180 degrees
- moved R15 34.4 mm to (117.1, 123.2)
- moved R16 33.8 mm to (117.1, 119.6), turned to 90 degrees
- moved R9 10.9 mm to (148.1, 116.4), turned to 90 degrees
- moved R6 9.84 mm to (144.7, 111.0), turned to 0 degrees
- moved R3 9.77 mm to (144.7, 109.8), turned to 180 degrees
- moved R10 7.48 mm to (150.9, 130.5), turned to 90 degrees
- moved R11 7.15 mm to (140.2, 130.0), turned to 0 degrees
- moved R7 6.49 mm to (144.7, 113.4), turned to 0 degrees
- moved R4 6.38 mm to (144.7, 112.2), turned to 180 degrees
- moved R8 3.84 mm to (144.7, 114.6), turned to 0 degrees
- moved R5 2.16 mm to (144.7, 115.8), turned to 180 degrees
- moved R1 0.60 mm to (144.7, 117.0), turned to 0 degrees
- renumbered R7 to R1, R18 to R17, R19 to R18, R1 to R3, R2 to R4, R3 to R5, R4 to R6, R5 to R7, R6 to R8
Connections:
- net /core-south-0/JTAG_TCK renamed /bridge/JTAG_TCK
- net /core-south-0/JTAG_TMS renamed /bridge/JTAG_TMS
- D1 pad 2: VCCO_0 -> +3V3
- J1 pad 2: VCCO_0 -> +3V3
- J1 pad 26: /core-south-0/CONFIG_CLK -> /config/CONFIG_CLK
- J1 pad 3: VCCO_0 -> +3V3
- J1 pad 4: VCCO_0 -> +3V3
- J1 pad 5: VCCO_0 -> +3V3
- J1 pad 59: /core-south-0/JTAG_TDO -> /bridge/JTAG_TDO
- J1 pad 60: /core-south-0/JTAG_TDI -> /bridge/JTAG_TDI
- J1 pad 86: VCCO_0 -> +3V3
- J1 pad 87: VCCO_0 -> +3V3
- J1 pad 88: VCCO_0 -> +3V3
- J1 pad 89: VCCO_0 -> +3V3
- J2 pad 2: VCCO_34 -> +3V3
- J2 pad 3: VCCO_34 -> +3V3
- J2 pad 4: VCCO_34 -> +3V3
- J2 pad 5: VCCO_34 -> +3V3
- J2 pad 86: VCCO_34 -> +3V3
- J2 pad 87: VCCO_34 -> +3V3
- J2 pad 88: VCCO_34 -> +3V3
- J2 pad 89: VCCO_34 -> +3V3
- J3 pad 2: VCCO_14 -> +3V3
- J3 pad 3: VCCO_14 -> +3V3
- J3 pad 4: VCCO_14 -> +3V3
- J3 pad 43: /core-north-14/IO14_1_P -> /config/CONFIG_MOSI_D00
- J3 pad 44: /core-north-14/IO14_1_N -> /config/CONFIG_DIN_D01
- J3 pad 5: VCCO_14 -> +3V3
- J3 pad 50: /core-north-14/IO14_2_N -> /config/CONFIG_D03
- J3 pad 51: /core-north-14/IO14_2_P -> /config/CONFIG_D02
- J3 pad 57: /core-north-14/IO14_6_P -> /config/CONFIG_FCS_B
- J3 pad 66: /core-north-14/IO14_12_P -> /config/CLK
- J3 pad 86: VCCO_14 -> +3V3
- J3 pad 87: VCCO_14 -> +3V3
- J3 pad 88: VCCO_14 -> +3V3
- J3 pad 89: VCCO_14 -> +3V3
- J4 pad 2: VCCO_15 -> +3V3
- J4 pad 3: VCCO_15 -> +3V3
- J4 pad 4: VCCO_15 -> +3V3
- J4 pad 5: VCCO_15 -> +3V3
- J4 pad 86: VCCO_15 -> +3V3
- J4 pad 87: VCCO_15 -> +3V3
- J4 pad 88: VCCO_15 -> +3V3
- J4 pad 89: VCCO_15 -> +3V3
- R1 pad 1: VCCO_0 -> +3V3
- R10 pad 2: VCCO_0 -> +3V3
- R11 pad 2: VCCO_0 -> +3V3
- R15 pad 2: VCCO_0 -> +3V3
- R16 pad 2: VCCO_0 -> +3V3
- R17 pad 2: VCCO_14 -> +3V3
- R3 pad 2: VCCO_0 -> +3V3
- R4 pad 2: VCCO_0 -> +3V3
- R5 pad 2: VCCO_0 -> +3V3
- R9 pad 2: VCCO_0 -> +3V3
Routing:
- net /config/CONFIG_CLK: track 0.00 -> 32.8 mm
- net /bridge/JTAG_TCK: track 0.00 -> 18.4 mm
- net /bridge/USB_DN: track 0.00 -> 16.5 mm
- net /bridge/USB_DP: track 0.00 -> 15.5 mm
- net /bridge/JTAG_TMS: track 0.00 -> 14.4 mm
- net /bridge/EECS: track 0.00 -> 12.4 mm
- net /bridge/EECLK: track 0.00 -> 10.6 mm
- net /core-south-0/CONFIG_M2: track 0.00 -> 10.5 mm
- net Net-(U4-OSCO): track 0.00 -> 9.20 mm
- net Net-(U4-OSCI): track 0.00 -> 8.79 mm
- net /core-south-0/CONFIG_M1: track 0.00 -> 7.96 mm
- net /power/EN_3V3: track 0.00 -> 7.53 mm, vias 0 -> 2
- net /bridge/EEDOUT: track 0.00 -> 6.40 mm
- net +3V3: track 0.00 -> 6.21 mm, vias 0 -> 19
- net /core-south-0/CONFIG_M0: track 0.00 -> 5.23 mm
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- added copper zone on F.Cu, net +1V8
- added copper zone on F.Cu, net +3V3
- added copper zone on In2.Cu, net +3V3
- added copper zone on F.Cu, net /bridge/VPHY
- added copper zone on F.Cu, net /bridge/VPLL
- added copper zone on F.Cu, net /power/SW_3V3
- added copper zone on B.Cu, net GND
- added copper zone on F.Cu, net GND
- added copper zone on In1.Cu, net GND
Other:
- board size 48 x 65 mm -> 100 x 60 mm
- board text added: "@supersmau"
- board text added: "June 2025"
- board text added: "Samuel López Asunción"
- board text added: "TCK"
- board text added: "TDI"
- board text added: "TDO"
- board text added: "TMS"
- board text added: "carrier.template.basic v1.0"
- board text added: "nuku.carrier.base"
- board text removed: "carrier.template.bare"

Commit message: Placement basic
Parts:
- moved SW2 103.1 mm to (174.9, 105.0)
- moved R43 98.2 mm to (173.5, 107.8), turned to 180 degrees
- moved R42 96.9 mm to (173.5, 102.2), turned to 180 degrees
- moved SW1 43.1 mm to (123.9, 121.0), turned to 90 degrees
- moved R11 18.0 mm to (150.5, 115.2), turned to 90 degrees
- moved R10 15.6 mm to (148.1, 115.2)
- moved R20 6.44 mm to (106.5, 116.2), turned to 90 degrees
- moved R19 6.10 mm to (107.7, 116.2), turned to -90 degrees
- moved L1 5.53 mm to (104.1, 120.2), turned to -90 degrees
- moved R21 4.49 mm to (110.9, 119.2), turned to 90 degrees
- moved R22 4.22 mm to (110.9, 121.2), turned to 90 degrees
- moved R15 4.12 mm to (113.5, 121.2), turned to 90 degrees
- moved R38 3.79 mm to (117.5, 114.2)
- moved C3 3.76 mm to (107.1, 123.0), turned to 0 degrees
- moved J6 3.62 mm to (117.5, 121.0)
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Routing:
- net +3V3: track 6.21 -> 19.7 mm, vias 19 -> 36
- net /config/CONFIG_CLK: track 32.8 -> 35.8 mm
- net /core-south-0/CONFIG_PROG: track 1.46 -> 3.75 mm
- net /core-south-0/CONFIG_DONE: track 2.79 -> 4.08 mm
- net Net-(D4-K): track 0.00 -> 1.29 mm
- net Net-(D3-K): track 0.00 -> 1.29 mm
- net Net-(D2-K): track 0.00 -> 1.29 mm
- net Net-(D1-K): track 0.00 -> 1.29 mm
- net /bridge/JTAG_TCK: track 18.4 -> 17.2 mm
- net /core-south-0/CONFIG_INIT: track 3.23 -> 4.25 mm
- net /core-south-0/CONFIG_M2: track 10.5 -> 11.5 mm
- net /core-south-0/CONFIG_M1: track 7.96 -> 8.72 mm
- net GND: vias 32 -> 65

Commit message: Finish template.basic + Production outputs
Parts:
- added 3V3: TestPoint_THTPad_D1.0mm_Drill0.5mm, TestPoint:TestPoint_THTPad_D1.0mm_Drill0.5mm, F.Cu at (103.9, 123.0)
- added 5VUSB: TestPoint_THTPad_D1.0mm_Drill0.5mm, TestPoint:TestPoint_THTPad_D1.0mm_Drill0.5mm, F.Cu at (102.5, 112.0)
- added GND: TestPoint_THTPad_D1.0mm_Drill0.5mm, TestPoint:TestPoint_THTPad_D1.0mm_Drill0.5mm, F.Cu at (103.9, 98.2)
- moved R41 21.1 mm to (120.5, 96.0), turned to 180 degrees
- moved C23 14.6 mm to (106.5, 87.2), turned to -90 degrees
- moved U5 13.9 mm to (121.9, 90.6), turned to 90 degrees
- moved U6 11.9 mm to (109.3, 87.8)
- moved R30 6.99 mm to (111.9, 91.6), turned to 180 degrees
- moved R32 6.71 mm to (111.9, 94.0), turned to 180 degrees
- moved R31 6.41 mm to (111.9, 92.8), turned to 180 degrees
- moved C22 5.37 mm to (118.1, 87.2), turned to -90 degrees
- moved C6 2.78 mm to (115.1, 88.8), turned to 0 degrees
- moved C15 1.00 mm to (110.7, 109.8)
- moved C10 0.40 mm to (109.7, 95.2)
- moved C21 0.20 mm to (117.5, 98.8)
Connections:
- ? pad 1: SHIELD -> (no net) (x4)
- J1 pad 32: /core-south-0/MGTP_CLK0_P -> /core-south-0/MGTP_CLK0_N
- J2 pad 47: /core-east-34/IO34_24_P -> /core-east-34/PMOD_A7
- J2 pad 48: /core-east-34/IO34_24_N -> /core-east-34/PMOD_A1
- J2 pad 50: /core-east-34/IO34_22_P -> /core-east-34/PMOD_A2
- J2 pad 51: /core-east-34/IO34_22_N -> /core-east-34/PMOD_A8
- J2 pad 53: /core-east-34/IO34_20_P -> /core-east-34/PMOD_A9
- J2 pad 54: /core-east-34/IO34_20_N -> /core-east-34/PMOD_A3
- J2 pad 56: /core-east-34/IO34_18_P -> /core-east-34/PMOD_A4
- J2 pad 57: /core-east-34/IO34_18_N -> /core-east-34/PMOD_A10
- J2 pad 68: /core-east-34/IO34_10_P -> /core-east-34/RESET
- J2 pad 71: /core-east-34/IO34_8_P -> /core-east-34/PMOD_B7
- J2 pad 72: /core-east-34/IO34_8_N -> /core-east-34/PMOD_B1
- J2 pad 74: /core-east-34/IO34_6_P -> /core-east-34/PMOD_B2
- J2 pad 75: /core-east-34/IO34_6_N -> /core-east-34/PMOD_B8
- J2 pad 77: /core-east-34/IO34_4_P -> /core-east-34/PMOD_B9
- J2 pad 78: /core-east-34/IO34_4_N -> /core-east-34/PMOD_B3
- J2 pad 80: /core-east-34/IO34_2_P -> /core-east-34/PMOD_B4
- J2 pad 81: /core-east-34/IO34_2_N -> /core-east-34/PMOD_B10
- J4 pad 62: /core-west-15/IO15_10_N -> /bridge/UART_TXD
- J4 pad 63: /core-west-15/IO15_10_P -> /bridge/UART_RXD
- J4 pad 65: /core-west-15/IO15_12_N -> /bridge/UART_RTS#
- J4 pad 66: /core-west-15/IO15_12_P -> /bridge/UART_CTS#
- J7 pad 1: /pmod/PMOD_A1 -> /core-east-34/PMOD_A1
- J7 pad 10: /pmod/PMOD_A10 -> /core-east-34/PMOD_A10
- J7 pad 2: /pmod/PMOD_A2 -> /core-east-34/PMOD_A2
- J7 pad 3: /pmod/PMOD_A3 -> /core-east-34/PMOD_A3
- J7 pad 4: /pmod/PMOD_A4 -> /core-east-34/PMOD_A4
- J7 pad 7: /pmod/PMOD_A7 -> /core-east-34/PMOD_A7
- J7 pad 8: /pmod/PMOD_A8 -> /core-east-34/PMOD_A8
- J7 pad 9: /pmod/PMOD_A9 -> /core-east-34/PMOD_A9
- J8 pad 1: /pmod/PMOD_B1 -> /core-east-34/PMOD_B1
- J8 pad 10: /pmod/PMOD_B10 -> /core-east-34/PMOD_B10
- J8 pad 2: /pmod/PMOD_B2 -> /core-east-34/PMOD_B2
- J8 pad 3: /pmod/PMOD_B3 -> /core-east-34/PMOD_B3
- J8 pad 4: /pmod/PMOD_B4 -> /core-east-34/PMOD_B4
- J8 pad 7: /pmod/PMOD_B7 -> /core-east-34/PMOD_B7
- J8 pad 8: /pmod/PMOD_B8 -> /core-east-34/PMOD_B8
- J8 pad 9: /pmod/PMOD_B9 -> /core-east-34/PMOD_B9
- R43 pad 1: /config/RESET -> /core-east-34/RESET
- U10 pad 1: /pmod/PMOD_B3 -> /core-east-34/PMOD_B3
- U10 pad 3: /pmod/PMOD_B4 -> /core-east-34/PMOD_B4
- U10 pad 4: /pmod/PMOD_B10 -> /core-east-34/PMOD_B10
- U10 pad 6: /pmod/PMOD_B9 -> /core-east-34/PMOD_B9
- U7 pad 1: /pmod/PMOD_A1 -> /core-east-34/PMOD_A1
- U7 pad 3: /pmod/PMOD_A2 -> /core-east-34/PMOD_A2
- U7 pad 4: /pmod/PMOD_A8 -> /core-east-34/PMOD_A8
- U7 pad 6: /pmod/PMOD_A7 -> /core-east-34/PMOD_A7
- U8 pad 1: /pmod/PMOD_B1 -> /core-east-34/PMOD_B1
- U8 pad 3: /pmod/PMOD_B2 -> /core-east-34/PMOD_B2
- U8 pad 4: /pmod/PMOD_B8 -> /core-east-34/PMOD_B8
- U8 pad 6: /pmod/PMOD_B7 -> /core-east-34/PMOD_B7
- U9 pad 1: /pmod/PMOD_A3 -> /core-east-34/PMOD_A3
- U9 pad 3: /pmod/PMOD_A4 -> /core-east-34/PMOD_A4
- U9 pad 4: /pmod/PMOD_A10 -> /core-east-34/PMOD_A10
- U9 pad 6: /pmod/PMOD_A9 -> /core-east-34/PMOD_A9
Routing:
- net /core-south-0/CONFIG_INIT: track 4.25 -> 70.6 mm, vias 1 -> 2
- net /bridge/JTAG_TDO: track 0.00 -> 57.6 mm, vias 0 -> 3
- net /bridge/JTAG_TDI: track 0.00 -> 52.3 mm, vias 0 -> 3
- net /config/CLK: track 0.00 -> 43.3 mm
- net /bridge/JTAG_TCK: track 17.2 -> 56.7 mm, vias 0 -> 2
- net /bridge/JTAG_TMS: track 14.5 -> 52.8 mm, vias 0 -> 2
- net /core-south-0/CONFIG_PROG: track 3.75 -> 37.6 mm, vias 1 -> 2
- net /config/CONFIG_FCS_B: track 2.01 -> 35.3 mm
- net /bridge/UART_RX_LED: track 4.20 -> 35.9 mm, vias 0 -> 2
- net /config/CONFIG_D03: track 0.00 -> 31.3 mm, vias 0 -> 2
- net /core-east-34/PMOD_B10: track 0.00 -> 29.2 mm
- net /config/CONFIG_D02: track 0.00 -> 27.8 mm
- net /config/CONFIG_CLK: track 35.8 -> 61.8 mm, vias 0 -> 2
- net /core-east-34/PMOD_B9: track 0.00 -> 25.9 mm
- net /core-east-34/PMOD_A7: track 0.00 -> 25.9 mm
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- added copper zone on In2.Cu, net +1V8
- added copper zone on F.Cu, net +5V
- added copper zone on In2.Cu, net +5V
- added copper zone on F.Cu, net /bridge/JTAG_VREF
- added copper zone on In2.Cu, net GND
- added copper zone on B.Cu, net SHIELD
Other:
- board text added: "0"
- board text added: "0 mm"
- board text added: "0.0152 mm"
- board text added: "0.02"
- board text added: "0.025 mm"
- board text added: "0.035 mm"
- board text added: "0.1000 mm / 0.1000 mm"
- board text added: "0.2104 mm"
- board text added: "0.2500 mm"
- board text added: "1"
- board text added: "1.065 mm"
- board text added: "1.6362 mm"
- board text added: "100.0000 mm x 60.0000 mm"
- board text added: "3.8"
- board text added: "4"
- board text added: "4.4"
- board text added: "4.6"
- board text added: "B.Mask"
- board text added: "B.Paste"
- board text added: "B.Silkscreen"
- board text added: "BOARD CHARACTERISTICS"
- board text added: "Board Thickness:"
- board text added: "Board overall dimensions:"
- board text added: "Bottom Silk Screen"
- board text added: "Bottom Solder Mask"
- board text added: "Bottom Solder Paste"
- board text added: "Castellated pads:"
- board text added: "Color"
- board text added: "Copper Finish:"
- board text added: "Copper Layer Count:"
- board text added: "Dielectric"
- board text added: "ENIG"
- board text added: "Edge card connectors:"
- board text added: "Epsilon R"
- board text added: "F.Mask"
- board text added: "F.Paste"
- board text added: "F.Silkscreen"
- board text added: "FR4"
- board text added: "FR4 natural"
- board text added: "FR4-7628"
- board text added: "Green"
- board text added: "Impedance Control:"
- board text added: "JLC"
- board text added: "L1_(Sig).Cu"
- board text added: "L2_(GND).Cu"
- board text added: "L3_(GND).Cu"
- board text added: "L4_(Sig).Cu"
- board text added: "Layer Name"
- board text added: "Liquid Photo"
- board text added: "Loss Tangent"
- board text added: "Material"
- board text added: "Min hole diameter:"
- board text added: "Min track/spacing:"
- board text added: "No"
- board text added: "Plated Board Edge:"
- board text added: "Thickness (mm)"
- board text added: "Top Silk Screen"
- board text added: "Top Solder Mask"
- board text added: "Top Solder Paste"
- board text added: "Type"
- board text added: "White"
- board text added: "Yes"
- board text added: "copper"
- board text added: "core"
- board text added: "nuku.carrier.template.basic"
- board text added: "prepreg"
- board text removed: "nuku.carrier.base"

Commit message: Finish bridgeless template
Parts:
- J6: footprint Connector:Tag-Connect_TC2050-IDC-NL_2x05_P1.27mm_Vertical -> Connector:Tag-Connect_TC2050-IDC-FP_2x05_P1.27mm_Vertical
- moved R21 2.00 mm to (110.9, 121.2), turned to -90 degrees
- moved R22 2.00 mm to (110.9, 119.2), turned to -90 degrees
