File: prj/nuku-carrier-template-basic/nuku-carrier-template-basic.kicad_pcb (KiCad board)
At the start: 4 copper layers, 100 x 60 mm, 91 parts, among them J1 DF40HC(4.0)-90DS-0.4V, J2 DF40HC(4.0)-90DS-0.4V, J3 DF40HC(4.0)-90DS-0.4V, J4 DF40HC(4.0)-90DS-0.4V, J5 USB_C_Receptacle_USB2.0_16P, J7 PMOD_A, J8 PMOD_B, SW1 PROG, SW2 RESET, U1 AP61302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

Commit message: Finish boards - prod ready
Parts:
- J1, J2, J3, J4: footprint nuku:DF40HC(4.0)-90DS-0.4V -> nuku:DF40C-90DS-0.4V
- moved R11 54.4 mm to (97.1, 125.6), turned to 180 degrees
- moved R10 34.7 mm to (114.3, 123.0)
- moved R17 33.0 mm to (110.3, 88.0), turned to 180 degrees
- moved R18 32.0 mm to (110.3, 86.8), turned to 0 degrees
- moved R1 28.0 mm to (116.7, 116.2), turned to -90 degrees
- moved R5 26.8 mm to (117.9, 116.2), turned to 90 degrees
- moved R8 25.6 mm to (119.1, 116.2), turned to -90 degrees
- moved R9 25.5 mm to (123.9, 112.6)
- moved R7 24.6 mm to (120.3, 116.2), turned to -90 degrees
- moved R4 23.5 mm to (121.5, 116.2), turned to 90 degrees
- moved R6 22.6 mm to (122.7, 116.2), turned to -90 degrees
- moved R3 21.8 mm to (123.9, 116.2), turned to 90 degrees
- moved R15 7.39 mm to (112.5, 116.2), turned to -90 degrees
- moved SW1 6.14 mm to (118.1, 123.0), turned to 180 degrees
- moved R16 4.42 mm to (114.7, 116.2), turned to -90 degrees
Routing:
- net /bridge/JTAG_TCK: track 0.00 -> 53.5 mm, vias 0 -> 2
- net /bridge/JTAG_TDI: track 0.00 -> 50.8 mm, vias 0 -> 2
- net /bridge/JTAG_TDO: track 0.00 -> 50.5 mm, vias 0 -> 2
- net /bridge/JTAG_TMS: track 0.03 -> 47.7 mm, vias 0 -> 2
- net /core-north-14/IO14_3_P: track 3.15 -> 37.4 mm, vias 0 -> 2
- net /core-south-0/CONFIG_CFGBVS: track 2.66 -> 31.6 mm
- net /core-south-0/CONFIG_DONE: track 4.08 -> 30.0 mm
- net /core-south-0/CONFIG_M0: track 5.52 -> 30.8 mm
- net /core-south-0/CONFIG_M1: track 8.72 -> 29.2 mm
- net /core-south-0/CONFIG_M2: track 11.5 -> 26.9 mm
- net /core-south-0/CONFIG_INIT: track 72.0 -> 67.3 mm
- net /core-south-0/CONFIG_PROG: track 43.5 -> 46.3 mm, vias 2 -> 0
- net /config/CONFIG_CLK: track 61.8 -> 59.0 mm
- net +3V3: track 21.8 -> 23.4 mm, vias 87 -> 86
- net GND: vias 237 -> 246
- added copper zone on In2.Cu, net GND
Other:
- board text removed: "Laboratorio de Sistemas Integrados DIE - ETSIT - UPM"
