File: prj/nuku-carrier-template-basic/usb.kicad_sch (KiCad schematic)
At the start: 8 parts, among them J5 USB_C_Receptacle_USB2.0_16P, U2 SRV05-4

Commit message: Route template.basic
Other:
- note added: "USB-C connector"
- moved on the sheet: R27
Changed lines of the file:
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@@
 		(comment 1 "@supersmau")
+	)
+	(rectangle
+		(start 81.28 57.15)
+		(end 219.71 146.05)
+		(stroke
+			(width 0)
+			(type dash)
+		)
+		(fill
+			(type none)
+		)
+	)
+	(rectangle
+		(start 200.66 118.11)
+		(end 214.63 125.73)
+		(stroke
+			(width 0)
+			(type dash)
+		)
+		(fill
+			(type none)
+		)
+	)
+	(text "USB-C connector"
+		(exclude_from_sim no)
+		(at 81.28 55.88 0)
+		(effects
+			(font
+				(size 1.27 1.27)
+				(italic yes)
+			)
+			(justify left bottom)
+		)
 	)
 	(junction
@@
 	)
 	(junction
-		(at 194.31 123.19)
+		(at 191.77 123.19)
 		(diameter 0)
 		(color 0 0 0 0)
@@
 	(wire
 		(pts
-			(xy 194.31 123.19) (xy 203.2 123.19)
+			(xy 191.77 123.19) (xy 203.2 123.19)
 		)
 		(stroke
@@
 	(wire
 		(pts
-			(xy 194.31 119.38) (xy 194.31 123.19)
+			(xy 191.77 119.38) (xy 191.77 123.19)
 		)
 		(stroke
@@
 	(wire
 		(pts
-			(xy 176.53 123.19) (xy 194.31 123.19)
+			(xy 176.53 123.19) (xy 191.77 123.19)
 		)
 		(stroke
@@
 	(wire
 		(pts
-			(xy 194.31 110.49) (xy 194.31 111.76)
+			(xy 191.77 110.49) (xy 191.77 111.76)
 		)
 		(stroke
@@
 	(symbol
 		(lib_id "power:VCC")
-		(at 194.31 110.49 0)
+		(at 191.77 110.49 0)
 		(unit 1)
 		(exclude_from_sim no)
@@
 		(fields_autoplaced yes)
 		(property "Reference" "#PWR055"
-			(at 194.31 114.3 0)
+			(at 191.77 114.3 0)
 			(effects
 				(font
@@
 		)
 		(property "Value" "+3V3"
-			(at 194.31 105.41 0)
+			(at 191.77 105.41 0)
 			(effects
 				(font
@@
 		)
 		(property "Footprint" ""
-			(at 194.31 110.49 0)
+			(at 191.77 110.49 0)
 			(effects
 				(font
@@
 		)
 		(property "Datasheet" ""
-			(at 194.31 110.49 0)
+			(at 191.77 110.49 0)
 			(effects
 				(font
@@
 		)
 		(property "Description" "Power symbol creates a global label with name \"VCC\""
-			(at 194.31 110.49 0)
+			(at 191.77 110.49 0)
 			(effects
 				(font
@@
 	(symbol
 		(lib_id "Device:R")
-		(at 194.31 115.57 180)
+		(at 191.77 115.57 180)
 		(unit 1)
 		(exclude_from_sim no)
 		(in_bom no)
-		(on_board yes)
+		(on_board no)
 		(dnp yes)
 		(property "Reference" "R27"
-			(at 196.85 114.2999 0)
+			(at 194.31 114.2999 0)
 			(effects
 				(font
@@
 		)
 		(property "Value" "1k5"
-			(at 196.85 116.8399 0)
+			(at 194.31 116.8399 0)
 			(effects
 				(font
@@
 		)
 		(property "Footprint" "Resistor_SMD:R_0402_1005Metric"
-			(at 196.088 115.57 90)
+			(at 193.548 115.57 90)
 			(effects
 				(font
@@
 		)
 		(property "Datasheet" "~"
-			(at 194.31 115.57 0)
+			(at 191.77 115.57 0)
 			(effects
 				(font
@@
 		)
 		(property "Description" "Resistor"
-			(at 194.31 115.57 0)
+			(at 191.77 115.57 0)
 			(effects
 				(font
@@
 		)
 		(property "LCSC" "C25867"
-			(at 194.31 115.57 0)
+			(at 191.77 115.57 0)
 			(effects
 				(font
@@
 		)
 		(property "Mfr. Part" ""
-			(at 194.31 115.57 0)
+			(at 191.77 115.57 0)
 			(effects
 				(font
@@
 		)
 		(property "Voltage" ""
-			(at 194.31 115.57 0)
-			(effects
-				(font
+			(at 191.77 115.57 0)
+			(effects
+				(font

Commit message: Finish bridgeless template
Other:
- moved on the sheet: R27, U2
