File: prj/nuku-carrier-template-basic/_autosave-nuku-carrier-template-basic.kicad_pcb (KiCad board)
At the start: 4 copper layers, 100 x 60 mm, 91 parts, among them J1 DF40HC(4.0)-90DS-0.4V, J2 DF40HC(4.0)-90DS-0.4V, J3 DF40HC(4.0)-90DS-0.4V, J4 DF40HC(4.0)-90DS-0.4V, J5 USB_C_Receptacle_USB2.0_16P, J7 PMOD_A, J8 PMOD_B, SW1 PROG, SW2 RESET, U1 AP61302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

Commit message: Tweaks
Parts:
- moved R11 54.4 mm to (97.1, 125.6), turned to 180 degrees
- moved R10 29.9 mm to (157.5, 143.6)
- moved R9 29.9 mm to (158.7, 143.6)
- moved R3 29.2 mm to (117.1, 119.4), turned to -90 degrees
- moved R6 27.7 mm to (118.3, 119.4), turned to 90 degrees
- moved R4 26.2 mm to (119.5, 119.4), turned to -90 degrees
- moved R7 24.7 mm to (120.7, 119.4), turned to 90 degrees
- moved R8 23.3 mm to (121.9, 119.4), turned to 90 degrees
- moved R15 22.2 mm to (137.7, 131.0)
- moved R16 22.2 mm to (137.7, 129.0)
- moved R5 21.9 mm to (123.1, 119.4), turned to -90 degrees
- moved R1 20.5 mm to (124.3, 119.4), turned to 90 degrees
- moved SW1 13.9 mm to (133.3, 131.2)
- moved R42 6.71 mm to (174.7, 108.8), turned to 0 degrees
- moved R43 2.78 mm to (172.1, 105.4), turned to -90 degrees
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Routing:
- net /core-south-0/CONFIG_DONE: track 4.08 -> 38.6 mm
- net /core-south-0/CONFIG_M2: track 11.5 -> 34.0 mm
- net /core-south-0/CONFIG_M1: track 8.72 -> 30.6 mm
- net /core-south-0/CONFIG_M0: track 5.52 -> 26.6 mm
- net /core-south-0/CONFIG_CFGBVS: track 2.66 -> 23.3 mm
- net /core-south-0/CONFIG_INIT: track 72.0 -> 86.2 mm, vias 2 -> 1
- net /core-south-0/CONFIG_PROG: track 43.5 -> 49.9 mm, vias 2 -> 1
- net /core-east-34/RESET: track 12.3 -> 6.11 mm
- net /bridge/JTAG_TCK: track 0.00 -> 5.28 mm
- net /bridge/JTAG_TDI: track 0.00 -> 4.30 mm
- net /bridge/JTAG_TDO: track 0.00 -> 4.10 mm
- net /bridge/JTAG_TMS: track 0.03 -> 3.83 mm
- net /config/CONFIG_CLK: track 61.8 -> 58.8 mm
- net /bridge/USB_DP: track 15.5 -> 16.2 mm
- net Net-(R42-Pad2): track 5.86 -> 6.42 mm
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