File: prj/nuku-carrier-template-basic/bridge.kicad_sch (KiCad schematic)
At the start: 33 parts, among them J6 TC2050, U3 FT93C46A-UTR-T, U4 FT2232HQ, Y1 12 MHz

Commit message: Route template.basic
Parts:
- added D3: RX, LED_SMD:LED_0805_2012Metric, symbol Device:LED
- added D4: TX, LED_SMD:LED_0805_2012Metric, symbol Device:LED
- added R36, R37: 1k, Resistor_SMD:R_0402_1005Metric, symbol Device:R
- U3: value FT93C46A-UTR-T -> M93C56-WDW6TP; LCSC C5263792 -> C2061074
- renumbered C15 to C10, C7 to C11, C7 to C12, C16 to C14, C8 to C15, C9 to C16, C8 to C17, C10 to C18, C9 to C19, C10 to C20, C11 to C21, C14 to C6, C6 to C7, C6 to C8, C12 to C9, L2 to L3, R36 to R39, R37 to R40
Connections:
- net AD0 is gone; now on net JTAG_TCK: U4.16 (ADBUS0)
- net AD1 is gone; now on net JTAG_TDI: U4.17 (ADBUS1)
- net AD2 is gone; now on net JTAG_TDO: U4.18 (ADBUS2)
- net AD3 is gone; now on net JTAG_TMS: U4.19 (ADBUS3)
- net +3V3: now also D3.2 (A), D4.2 (A)
- net JTAG_TCK: no longer U4.38 (BDBUS0)
- net JTAG_TDI: no longer U4.39 (BDBUS1)
- net JTAG_TDO: no longer U4.40 (BDBUS2)
- net JTAG_TMS: no longer U4.41 (BDBUS3)
- net UART_RX_LED: now reaches U4.54 (BCBUS3)
- net UART_RX_LED: now also R36.1
- net UART_TX_LED: now reaches U4.55 (BCBUS4)
- net UART_TX_LED: now also R37.1
- net AC0: no longer names the net of U4.26 (ACBUS0)
- net AC1: no longer names the net of U4.27 (ACBUS1)
- net AC2: no longer names the net of U4.28 (ACBUS2)
- net AC3: no longer names the net of U4.29 (ACBUS3)
- net AC4: no longer names the net of U4.30 (ACBUS4)
- net AC5: no longer names the net of U4.32 (ACBUS5)
- net AC6: no longer names the net of U4.33 (ACBUS6)
- net AC7: no longer names the net of U4.34 (ACBUS7)
- net AD4: no longer names the net of U4.21 (ADBUS4)
- net AD5: no longer names the net of U4.22 (ADBUS5)
- net AD6: no longer names the net of U4.23 (ADBUS6)
- net AD7: no longer names the net of U4.24 (ADBUS7)
- new net: D4.1 (K), R37.2
- new net: D3.1 (K), R36.2
- new net UART_CTS#: U4.41 (BDBUS3)
- new net UART_RTS#: U4.40 (BDBUS2)
- new net UART_RXD: U4.39 (BDBUS1)
- new net UART_TXD: U4.38 (BDBUS0)
- no-connect marks 12 -> 21
Other:
- note added: "Dual USB-to-JTAG/UART bridge"
- note removed: "CTS#"
- note removed: "RTS#"
- note removed: "RXD"
- note removed: "RXLED#"
- note removed: "TXD"
- note removed: "TXLED#"
- moved on the sheet: C10, C11, C12, C13, C14, C15, C16, C17, C18, C19, C20, C21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

Commit message: Finish template.basic + Production outputs
Connections:
- no-connect marks 21 -> 22
Changed lines of the file:
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@@
+	)
+	(no_connect
+		(at 269.24 59.69)
 	)
 	(no_connect

Commit message: Finish bridgeless template
Parts:
- J6: footprint Connector:Tag-Connect_TC2050-IDC-NL_2x05_P1.27mm_Vertical -> Connector:Tag-Connect_TC2050-IDC-FP_2x05_P1.27mm_Vertical
- U3: value M93C56-WDW6TP -> M93C56-WMN6TP; footprint Package_SO:TSSOP-8_4.4x3mm_P0.65mm -> Package_SO:SOIC-8_3.9x4.9mm_P1.27mm; LCSC C2061074 -> C283453
Connections:
- net PWREN: no longer names the net of U4.60 (~{PWREN})
- net SUSPEND: no longer names the net of U4.36 (~{SUSPEND})
- no-connect marks 22 -> 24
Changed lines of the file:
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@@
 	)
 	(rectangle
-		(start 195.58 66.04)
+		(start 198.12 66.04)
 		(end 209.55 71.12)
 		(stroke
@@
 	)
 	(rectangle
-		(start 195.58 99.06)
+		(start 198.12 99.06)
 		(end 209.55 104.14)
 		(stroke
@@
 	)
 	(rectangle
-		(start 179.07 147.32)
-		(end 193.04 154.94)
-		(stroke
-			(width 0)
-			(type dash)
-		)
-		(fill
-			(type none)
-		)
-	)
-	(rectangle
 		(start 50.8 81.28)
 		(end 64.77 88.9)
@@
 	)
 	(no_connect
+		(at 179.07 152.4)
+	)
+	(no_connect
+		(at 179.07 149.86)
+	)
+	(no_connect
 		(at 179.07 86.36)
 	)
@@
 	(wire
 		(pts
-			(xy 180.34 149.86) (xy 179.07 149.86)
-		)
-		(stroke
-			(width 0)
-			(type default)
-		)
-	)
-	(wire
-		(pts
 			(xy 218.44 121.92) (xy 218.44 124.46)
 		)
@@
 	(wire
 		(pts
-			(xy 180.34 152.4) (xy 179.07 152.4)
-		)
-		(stroke
-			(width 0)
-			(type default)
-		)
-	)
-	(wire
-		(pts
 			(xy 228.6 59.69) (xy 243.84 59.69)
 		)
@@
 		)
 	)
-	(hierarchical_label "PWREN"
-		(shape output)
-		(at 180.34 149.86 0)
-		(effects
-			(font
-				(size 1.27 1.27)
-			)
-			(justify left)
-		)
-	)
 	(hierarchical_label "{JTAG}"
 		(shape bidirectional)
@@
 		)
 	)
-	(hierarchical_label "SUSPEND"
-		(shape output)
-		(at 180.34 152.4 0)
-		(effects
-			(font
-				(size 1.27 1.27)
-			)
-			(justify left)
-		)
-	)
 	(symbol
 		(lib_id "Memory_EEPROM:93CxxC")
@@
 			)
 		)
-		(property "Value" "M93C56-WDW6TP"
+		(property "Value" "M93C56-WMN6TP"
 			(at 52.9941 119.38 0)
 			(effects
@@
 			)
 		)
-		(property "Footprint" "Package_SO:TSSOP-8_4.4x3mm_P0.65mm"
+		(property "Footprint" "Package_SO:SOIC-8_3.9x4.9mm_P1.27mm"
 			(at 50.8 127 0)
 			(effects
@@
 			)
 		)
-		(property "Datasheet" "https://jlcpcb.com/api/file/downloadByFileSystemAccessId/8588932626149756928"
+		(property "Datasheet" "https://jlcpcb.com/api/file/downloadByFileSystemAccessId/8588904334871941120"
 			(at 50.8 127 0)
 			(effects
@@
 			)
 		)
-		(property "LCSC" "C2061074"
+		(property "LCSC" "C283453"
 			(at 50.8 127 0)
 			(effects
@@
 			)
 		)
-		(property "Footprint" "Connector:Tag-Connect_TC2050-IDC-NL_2x05_P1.27mm_Vertical"
+		(property "Footprint" "Connector:Tag-Connect_TC2050-IDC-FP_2x05_P1.27mm_Vertical"
 			(at 250.19 64.77 0)
 			(effects

Commit message: Tweaks
Parts:
- removed J6: TC2050, Connector:Tag-Connect_TC2050-IDC-FP_2x05_P1.27mm_Vertical, symbol Connector:TC2050
- removed R38: 0, Resistor_SMD:R_0402_1005Metric, symbol Device:R
Connections:
- no-connect marks 24 -> 23
Other:
- note removed: "JTAG"
- note removed: "Pin 1 (VREF) drives the programmer's output drivers Draws ~ 10 mA @ +3V3"
- note removed: "See Tag-Connect TC2050-Xilinx Adaptor Sheet"
- note removed: "See Xilinx Platform Cable USB II (DS593)"
- moved on the sheet: C10, C11, C12, C13, C14, C15, C16, C17, C18, C19, C20, C21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
