File: prj/nuku-carrier-template-basic/core-south.kicad_sch (KiCad schematic)
At the start: 19 parts, among them J1 DF40HC(4.0)-90DS-0.4V, SW1 PROG

Commit message: Finish boards - prod ready
Parts:
- J1: footprint nuku:DF40HC(4.0)-90DS-0.4V -> nuku:DF40C-90DS-0.4V; symbol nuku:DF40HC(4.0)-90DS-0.4V -> nuku:DF40C-90DS-0.4V; LCSC C597947 -> C2911197
Changed lines of the file:
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@@
 	)
 	(symbol
-		(lib_name "DF40HC(4.0)-90DS-0.4V_1")
-		(lib_id "nuku:DF40HC(4.0)-90DS-0.4V")
+		(lib_id "nuku:DF40C-90DS-0.4V")
 		(at 223.52 39.37 0)
 		(unit 1)
@@
 			)
 		)
-		(property "Footprint" "nuku:DF40HC(4.0)-90DS-0.4V"
+		(property "Footprint" "nuku:DF40C-90DS-0.4V"
 			(at 223.52 156.21 0)
 			(effects
@@
 			)
 		)
-		(property "Datasheet" "https://www.lcsc.com/datasheet/lcsc_datasheet_2006112253_HRS-Hirose-DF40HC-4-0-90DS-0-4V-51_C597947.pdf"
+		(property "Datasheet" "https://www.lcsc.com/datasheet/lcsc_datasheet_2206011716_HRS-Hirose-DF40C-90DS-0-4V-51_C2911197.pdf"
 			(at 223.52 158.75 0)
 			(effects
@@
 			)
 		)
-		(property "LCSC" "C597947"
-			(at 223.52 39.37 0)
+		(property "LCSC" "C2911197"
+			(at 223.52 160.02 0)
 			(effects
 				(font
 					(size 1.27 1.27)
 				)
+				(justify left top)
 				(hide yes)
 			)
