File: prj/nuku-carrier-template-bridgeless/config.kicad_sch (KiCad schematic)
At the start: 5 parts, among them U5 IS25LP064A, U6 OT3225100MJBA4SL

Commit message: Finish bridgeless template
Parts:
- renumbered C22 to C6, C23 to C7, R41 to R28, U5 to U2, U6 to U3
Changed lines of the file:
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@@
 	(title_block
 		(title "nuku.carrier.template.basic")
-		(date "2025-06-09")
+		(date "2025-06-28")
 		(rev "0")
 		(company "Samuel López Asunción")
@@
 		(on_board yes)
 		(dnp no)
-		(property "Reference" "#PWR048"
+		(property "Reference" "#PWR038"
 			(at 143.51 125.73 0)
 			(effects
@@
 			(project "nuku-carrier-template-basic"
 				(path "/15e0a42f-48e0-4a5d-9b6b-7d249ffc02ad/7dac40ed-a7ca-4544-9148-bf95ff4c6d66"
-					(reference "#PWR048")
+					(reference "#PWR038")
 					(unit 1)
 				)
@@
 		(on_board yes)
 		(dnp no)
-		(property "Reference" "C23"
+		(property "Reference" "C7"
 			(at 170.18 109.2199 0)
 			(effects
@@
 			(project "nuku-carrier-template-basic"
 				(path "/15e0a42f-48e0-4a5d-9b6b-7d249ffc02ad/7dac40ed-a7ca-4544-9148-bf95ff4c6d66"
-					(reference "C23")
+					(reference "C7")
 					(unit 1)
 				)
@@
 		(on_board yes)
 		(dnp no)
-		(property "Reference" "#PWR049"
+		(property "Reference" "#PWR039"
 			(at 173.99 109.22 0)
 			(effects
@@
 			(project "nuku-carrier-template-basic"
 				(path "/15e0a42f-48e0-4a5d-9b6b-7d249ffc02ad/7dac40ed-a7ca-4544-9148-bf95ff4c6d66"
-					(reference "#PWR049")
+					(reference "#PWR039")
 					(unit 1)
 				)
@@
 		(on_board yes)
 		(dnp no)
-		(property "Reference" "#PWR050"
+		(property "Reference" "#PWR040"
 			(at 173.99 121.92 0)
 			(effects
@@
 			(project "nuku-carrier-template-basic"
 				(path "/15e0a42f-48e0-4a5d-9b6b-7d249ffc02ad/7dac40ed-a7ca-4544-9148-bf95ff4c6d66"
-					(reference "#PWR050")
+					(reference "#PWR040")
 					(unit 1)
 				)
@@
 		(dnp no)
 		(fields_autoplaced yes)
-		(property "Reference" "U5"
+		(property "Reference" "U2"
 			(at 129.54 95.25 0)
 			(effects
@@
 			(project "nuku-carrier-template-basic"
 				(path "/15e0a42f-48e0-4a5d-9b6b-7d249ffc02ad/7dac40ed-a7ca-4544-9148-bf95ff4c6d66"
-					(reference "U5")
+					(reference "U2")
 					(unit 1)
 				)
@@
 		(on_board yes)
 		(dnp no)
-		(property "Reference" "#PWR046"
+		(property "Reference" "#PWR036"
 			(at 115.57 95.25 0)
 			(effects
@@
 			(project "nuku-carrier-template-basic"
 				(path "/15e0a42f-48e0-4a5d-9b6b-7d249ffc02ad/7dac40ed-a7ca-4544-9148-bf95ff4c6d66"
-					(reference "#PWR046")
+					(reference "#PWR036")
 					(unit 1)
 				)
@@
 		(on_board yes)
 		(dnp no)
-		(property "Reference" "#PWR047"
+		(property "Reference" "#PWR037"
 			(at 143.51 105.41 0)
 			(effects
@@
 			(project "nuku-carrier-template-basic"
 				(path "/15e0a42f-48e0-4a5d-9b6b-7d249ffc02ad/7dac40ed-a7ca-4544-9148-bf95ff4c6d66"
-					(reference "#PWR047")
+					(reference "#PWR037")
 					(unit 1)
 				)
@@
 		(dnp no)
 		(fields_autoplaced yes)
-		(property "Reference" "U6"
+		(property "Reference" "U3"
 			(at 189.23 99.06 0)
 			(effects
@@
 			(project "nuku-carrier-template-basic"
 				(path "/15e0a42f-48e0-4a5d-9b6b-7d249ffc02ad/7dac40ed-a7ca-4544-9148-bf95ff4c6d66"
-					(reference "U6")
+					(reference "U3")
 					(unit 1)
 				)
@@
 		(on_board yes)
 		(dnp no)
-		(property "Reference" "R41"
+		(property "Reference" "R28"
 			(at 109.22 95.25 0)
 			(effects
@@
 			(project "nuku-carrier-template-basic"
 				(path "/15e0a42f-48e0-4a5d-9b6b-7d249ffc02ad/7dac40ed-a7ca-4544-9148-bf95ff4c6d66"
-					(reference "R41")
+					(reference "R28")
 					(unit 1)
 				)
@@
 		(dnp no)
 		(fields_autoplaced yes)
-		(property "Reference" "C22"
+		(property "Reference" "C6"
 			(at 147.32 109.2199 0)
 			(effects
@@
 			(project "nuku-carrier-template-basic"
 				(path "/15e0a42f-48e0-4a5d-9b6b-7d249ffc02ad/7dac40ed-a7ca-4544-9148-bf95ff4c6d66"
-					(reference "C22")
+					(reference "C6")
 					(unit 1)
 				)
