File: prj/nuku-carrier-template-bridgeless/core-east.kicad_sch (KiCad schematic)
At the start: 1 part, among them J4 DF40HC(4.0)-90DS-0.4V

Commit message: Finish bridgeless template
Parts:
- removed J4: DF40HC(4.0)-90DS-0.4V, nuku:DF40HC(4.0)-90DS-0.4V, symbol nuku:DF40HC(4.0)-90DS-0.4V
- added J2: DF40C-90DS-0.4V, nuku:DF40C-90DS-0.4V, symbol nuku:DF40C-90DS-0.4V
Connections:
- net GND: now also J2.1, J2.12, J2.15, J2.18, J2.21, J2.24, J2.27, J2.30, J2.33, J2.36, J2.39, J2.42, J2.44, J2.45, J2.46, J2.49, J2.52, J2.55, J2.58, J2.6, J2.61, J2.64, J2.67, J2.70, J2.73, J2.76, J2.79, J2.82, J2.84, J2.85, J2.9, J2.90
- new net IO34_0: J2.83
- new net IO34_10_N: J2.69
- new net IO34_11_N: J2.22
- new net IO34_11_P: J2.23
- new net IO34_12_N: J2.66
- new net IO34_12_P: J2.65
- new net IO34_13_N: J2.25
- new net IO34_13_P: J2.26
- new net IO34_14_N: J2.63
- new net IO34_14_P: J2.62
- new net IO34_15_N: J2.28
- new net IO34_15_P: J2.29
- new net IO34_16_N: J2.60
- new net IO34_16_P: J2.59
- new net IO34_17_N: J2.31
- new net IO34_17_P: J2.32
- new net IO34_19_N: J2.34
- new net IO34_19_P: J2.35
- new net IO34_1_N: J2.7
- new net IO34_1_P: J2.8
- new net IO34_21_N: J2.37
- new net IO34_21_P: J2.38
- new net IO34_23_N: J2.40
- new net IO34_23_P: J2.41
- new net IO34_25: J2.43
- new net IO34_3_N: J2.10
- new net IO34_3_P: J2.11
- new net IO34_5_N: J2.13
- new net IO34_5_P: J2.14
- new net IO34_7_N: J2.16
- new net IO34_7_P: J2.17
- new net IO34_9_N: J2.19
- new net IO34_9_P: J2.20
- new net PMOD_A1: J2.48
- new net PMOD_A10: J2.57
- new net PMOD_A2: J2.50
- new net PMOD_A3: J2.54
- new net PMOD_A4: J2.56
- new net PMOD_A7: J2.47
- new net PMOD_A8: J2.51
- new net PMOD_A9: J2.53
- new net PMOD_B1: J2.72
- new net PMOD_B10: J2.81
- new net PMOD_B2: J2.74
- new net PMOD_B3: J2.78
- new net PMOD_B4: J2.80
- new net PMOD_B7: J2.71
- new net PMOD_B8: J2.75
- new net PMOD_B9: J2.77
- new net RESET: J2.68
- new net VCCO_34: J2.2, J2.3, J2.4, J2.5, J2.86, J2.87, J2.88, J2.89
- no-connect marks 46 -> 33
