File: prj/nuku-carrier-template-bridgeless/core-north.kicad_sch (KiCad schematic)
At the start: 1 part, among them J4 DF40HC(4.0)-90DS-0.4V

Commit message: Finish bridgeless template
Parts:
- removed J4: DF40HC(4.0)-90DS-0.4V, nuku:DF40HC(4.0)-90DS-0.4V, symbol nuku:DF40HC(4.0)-90DS-0.4V
- added J3: DF40C-90DS-0.4V, nuku:DF40C-90DS-0.4V, symbol nuku:DF40C-90DS-0.4V
- added R17, R18: 1k, Resistor_SMD:R_0402_1005Metric, symbol Device:R
Connections:
- net GND: now also J3.1, J3.12, J3.15, J3.18, J3.21, J3.24, J3.27, J3.30, J3.33, J3.36, J3.39, J3.42, J3.45, J3.46, J3.47, J3.49, J3.52, J3.55, J3.58, J3.6, J3.61, J3.64, J3.67, J3.7, J3.70, J3.73, J3.76, J3.79, J3.82, J3.85, J3.9, J3.90, R18.1
- new net CLK: J3.66
- new net CONFIG_D02: J3.51
- new net CONFIG_D03: J3.50
- new net CONFIG_DIN_D01: J3.44
- new net CONFIG_FCS_B: J3.57
- new net CONFIG_MOSI_D00: J3.43
- new net IO14_0: J3.48
- new net IO14_10_N: J3.62
- new net IO14_10_P: J3.63
- new net IO14_11_N: J3.29
- new net IO14_11_P: J3.28
- new net IO14_12_N: J3.65
- new net IO14_13_N: J3.26
- new net IO14_13_P: J3.25
- new net IO14_14_N: J3.68
- new net IO14_14_P: J3.69
- new net IO14_15_N: J3.23
- new net IO14_15_P: J3.22
- new net IO14_16_N: J3.71
- new net IO14_16_P: J3.72
- new net IO14_17_N: J3.20
- new net IO14_17_P: J3.19
- new net IO14_18_N: J3.74
- new net IO14_18_P: J3.75
- new net IO14_19_N: J3.17
- new net IO14_19_P: J3.16
- new net IO14_20_N: J3.77
- new net IO14_20_P: J3.78
- new net IO14_21_N: J3.14
- new net IO14_21_P: J3.13
- new net IO14_22_N: J3.80
- new net IO14_22_P: J3.81
- new net IO14_23_N: J3.11
- new net IO14_23_P: J3.10
- new net IO14_24_N: J3.83
- new net IO14_24_P: J3.84
- new net IO14_25: J3.8
- new net IO14_3_N: J3.41
- new net IO14_3_P: J3.40, R17.1, R18.2
- new net IO14_4_N: J3.53
- new net IO14_4_P: J3.54
- new net IO14_5_N: J3.38
- new net IO14_5_P: J3.37
- new net IO14_6_N: J3.56
- new net IO14_7_N: J3.35
- new net IO14_7_P: J3.34
- new net IO14_8_N: J3.59
- new net IO14_8_P: J3.60
- new net IO14_9_N: J3.32
- new net IO14_9_P: J3.31
- new net VCCO_14: J3.2, J3.3, J3.4, J3.5, J3.86, J3.87, J3.88, J3.89, R17.2
- no-connect marks 46 -> 43
Other:
- note added: "CLK -> IO_L12P_T1_MRCC_14 Multi-region clock"
- note added: "CONFIG_PUDC_B"
