File: prj/nuku-carrier-template-bridgeless/core-west.kicad_sch (KiCad schematic)
At the start: 1 part, among them J4 DF40HC(4.0)-90DS-0.4V

Commit message: Finish bridgeless template
Parts:
- J4: value DF40HC(4.0)-90DS-0.4V -> DF40C-90DS-0.4V; footprint nuku:DF40HC(4.0)-90DS-0.4V -> nuku:DF40C-90DS-0.4V; symbol nuku:DF40HC(4.0)-90DS-0.4V -> nuku:DF40C-90DS-0.4V; LCSC C597947 -> C2911197
Connections:
- net UART_CTS# renamed IO15_12_P
- net UART_RTS# renamed IO15_12_N
- net UART_RXD renamed IO15_10_P
- net UART_TXD renamed IO15_10_N
- no-connect marks 46 -> 50
Changed lines of the file:
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@@
 	(title_block
 		(title "nuku.carrier.template.basic")
-		(date "2025-06-09")
+		(date "2025-06-28")
 		(rev "0")
 		(company "Samuel López Asunción")
 		(comment 1 "@supersmau")
 	)
-	(rectangle
-		(start 186.69 96.52)
-		(end 198.12 101.6)
-		(stroke
-			(width 0)
-			(type dash)
-		)
-		(fill
-			(type none)
-		)
-	)
 	(junction
 		(at 163.83 48.26)
@@
 	)
 	(no_connect
+		(at 182.88 101.6)
+	)
+	(no_connect
 		(at 114.3 73.66)
 	)
@@
 	)
 	(no_connect
+		(at 182.88 109.22)
+	)
+	(no_connect
 		(at 182.88 134.62)
 	)
@@
 	)
 	(no_connect
+		(at 182.88 104.14)
+	)
+	(no_connect
 		(at 114.3 78.74)
 	)
@@
 	)
 	(no_connect
+		(at 182.88 111.76)
+	)
+	(no_connect
 		(at 114.3 127)
 	)
@@
 		(at 114.3 132.08)
 	)
-	(bus_entry
-		(at 182.88 111.76)
-		(size 2.54 -2.54)
-		(stroke
-			(width 0)
-			(type default)
-		)
-	)
-	(bus_entry
-		(at 185.42 106.68)
-		(size -2.54 2.54)
-		(stroke
-			(width 0)
-			(type default)
-		)
-	)
-	(bus_entry
-		(at 185.42 99.06)
-		(size -2.54 2.54)
-		(stroke
-			(width 0)
-			(type default)
-		)
-	)
-	(bus_entry
-		(at 185.42 101.6)
-		(size -2.54 2.54)
-		(stroke
-			(width 0)
-			(type default)
-		)
-	)
 	(wire
 		(pts
@@
 		)
 	)
-	(bus
-		(pts
-			(xy 185.42 101.6) (xy 185.42 99.06)
-		)
-		(stroke
-			(width 0)
-			(type default)
-		)
-	)
 	(wire
 		(pts
@@
 		)
 	)
-	(bus
-		(pts
-			(xy 185.42 99.06) (xy 187.96 99.06)
-		)
-		(stroke
-			(width 0)
-			(type default)
-		)
-	)
 	(wire
 		(pts
@@
 		)
 	)
-	(bus
-		(pts
-			(xy 185.42 109.22) (xy 185.42 106.68)
-		)
-		(stroke
-			(width 0)
-			(type default)
-		)
-	)
 	(wire
 		(pts
@@
 		(pts
 			(xy 154.94 86.36) (xy 182.88 86.36)
-		)
-		(stroke
-			(width 0)
-			(type default)
-		)
-	)
-	(bus
-		(pts
-			(xy 185.42 106.68) (xy 185.42 101.6)
 		)
 		(stroke
@@
 		)
 	)
-	(label "UART_CTS#"
-		(at 182.88 101.6 180)
-		(effects
-			(font
-				(size 1.27 1.27)
-			)
-			(justify right bottom)
-		)
-	)
 	(label "IO15_23_N"
 		(at 114.3 66.04 0)
@@
 		)
 	)
-	(label "UART_TXD"
-		(at 182.88 111.76 180)
+	(label "IO15_10_P"
+		(at 182.88 109.22 180)
 		(effects
 			(font
@@
 			)
 			(justify right bottom)
+		)
+		(property "Netclass" "DIFF_92"
+			(at 161.29 109.22 0)
+			(effects
+				(font
+					(size 1.27 1.27)
+					(italic yes)
+				)
+				(justify left bottom)
+			)
 		)
 	)
@@
 		)
 	)
-	(label "UART_RTS#"
-		(at 182.88 104.14 180)
-		(effects
-			(font
-				(size 1.27 1.27)
-			)
-			(justify right bottom)
-		)
-	)
 	(label "IO15_18_N"
 		(at 182.88 81.28 180)
@@
 		)
 	)
+	(label "IO15_12_P"
+		(at 182.88 101.6 180)
+		(effects
+			(font
+				(size 1.27 1.27)
+			)
+			(justify right bottom)
+		)
+		(property "Netclass" "DIFF_92"
+			(at 161.29 101.6 0)
+			(effects
+				(font
+					(size 1.27 1.27)
+					(italic yes)
+				)
+				(justify left bottom)
+			)
+		)
+	)
 	(label "IO15_16_P"
 		(at 182.88 86.36 180)
@@
 		)
 	)
-	(label "UART_RXD"
-		(at 182.88 109.22 180)
-		(effects
-			(font
-				(size 1.27 1.27)
-			)
-			(justify right bottom)
-		)
-	)
 	(label "IO15_0"
 		(at 182.88 147.32 180)
@@
 		)
 	)
+	(label "IO15_10_N"
+		(at 182.88 111.76 180)
+		(effects
+			(font
+				(size 1.27 1.27)
+			)
+			(justify right bottom)
+		)
+		(property "Netclass" "DIFF_92"
+			(at 161.29 111.76 0)
+			(effects
+				(font
+					(size 1.27 1.27)
+					(italic yes)
+				)
+				(justify left bottom)
+			)
+		)
+	)
 	(label "IO15_3_P"
 		(at 114.3 139.7 0)
@@
 		)
 	)
+	(label "IO15_12_N"
+		(at 182.88 104.14 180)
+		(effects
+			(font
+				(size 1.27 1.27)
+			)
+			(justify right bottom)
+		)
+		(property "Netclass" "DIFF_92"
+			(at 161.29 104.14 0)
+			(effects
+				(font
+					(size 1.27 1.27)
+					(italic yes)
+				)
+				(justify left bottom)
+			)
+		)
+	)
 	(label "IO15_17_N"
 		(at 114.3 88.9 0)
@@
 				(justify right bottom)
 			)
-		)
-	)
-	(hierarchical_label "{UART}"
-		(shape bidirectional)
-		(at 187.96 99.06 0)
-		(effects
-			(font
-				(size 1.27 1.27)
-			)
-			(justify left)
 		)
 	)
@@
 	)
 	(symbol
-		(lib_id "nuku:DF40HC(4.0)-90DS-0.4V")
+		(lib_id "nuku:DF40C-90DS-0.4V")
 		(at 146.05 39.37 0)
 		(unit 1)
@@
 			)
 		)
-		(property "Value" "DF40HC(4.0)-90DS-0.4V"
+		(property "Value" "DF40C-90DS-0.4V"
 			(at 148.59 36.83 0)
 			(effects
@@
 			)
 		)
-		(property "Footprint" "nuku:DF40HC(4.0)-90DS-0.4V"
+		(property "Footprint" "nuku:DF40C-90DS-0.4V"
 			(at 146.05 156.21 0)
 			(effects
@@
 			)
 		)
-		(property "Datasheet" "https://www.lcsc.com/datasheet/lcsc_datasheet_2006112253_HRS-Hirose-DF40HC-4-0-90DS-0-4V-51_C597947.pdf"
+		(property "Datasheet" "https://www.lcsc.com/datasheet/lcsc_datasheet_2206011716_HRS-Hirose-DF40C-90DS-0-4V-51_C2911197.pdf"
 			(at 146.05 158.75 0)
 			(effects
@@
 			)
 		)
-		(property "LCSC" "C597947"
+		(property "LCSC" "C2911197"
 			(at 146.05 39.37 0)
 			(effects
