File: prj/nuku-carrier-template-bridgeless/pmod.kicad_sch (KiCad schematic)
At the start: 9 parts, among them J7 PMOD_A, J8 PMOD_B, SW2 RESET, U10 SRV05-4, U7 SRV05-4, U8 SRV05-4, U9 SRV05-4

Commit message: Finish bridgeless template
Parts:
- renumbered R42 to R29, R43 to R30, U7 to U4, U8 to U5, U9 to U6, U10 to U7
Changed lines of the file:
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@@
 	(title_block
 		(title "nuku.carrier.template.basic")
-		(date "2025-06-09")
+		(date "2025-06-28")
 		(rev "0")
 		(company "Samuel López Asunción")
@@
 		(on_board yes)
 		(dnp no)
-		(property "Reference" "#PWR071"
+		(property "Reference" "#PWR053"
 			(at 167.64 93.98 0)
 			(effects
@@
 			(project "nuku-carrier-template-basic"
 				(path "/15e0a42f-48e0-4a5d-9b6b-7d249ffc02ad/cb35697b-7148-4b12-9d2d-66ae29597163"
-					(reference "#PWR071")
+					(reference "#PWR053")
 					(unit 1)
 				)
@@
 		(on_board yes)
 		(dnp no)
-		(property "Reference" "#PWR051"
+		(property "Reference" "#PWR043"
 			(at 91.44 73.66 0)
 			(effects
@@
 			(project "nuku-carrier-template-basic"
 				(path "/15e0a42f-48e0-4a5d-9b6b-7d249ffc02ad/cb35697b-7148-4b12-9d2d-66ae29597163"
-					(reference "#PWR051")
+					(reference "#PWR043")
 					(unit 1)
 				)
@@
 		(on_board yes)
 		(dnp no)
-		(property "Reference" "#PWR064"
+		(property "Reference" "#PWR046"
 			(at 93.98 121.92 0)
 			(effects
@@
 			(project "nuku-carrier-template-basic"
 				(path "/15e0a42f-48e0-4a5d-9b6b-7d249ffc02ad/cb35697b-7148-4b12-9d2d-66ae29597163"
-					(reference "#PWR064")
+					(reference "#PWR046")
 					(unit 1)
 				)
@@
 		(on_board yes)
 		(dnp no)
-		(property "Reference" "#PWR061"
+		(property "Reference" "#PWR044"
 			(at 91.44 118.11 0)
 			(effects
@@
 			(project "nuku-carrier-template-basic"
 				(path "/15e0a42f-48e0-4a5d-9b6b-7d249ffc02ad/cb35697b-7148-4b12-9d2d-66ae29597163"
-					(reference "#PWR061")
+					(reference "#PWR044")
 					(unit 1)
 				)
@@
 		(on_board yes)
 		(dnp no)
-		(property "Reference" "#PWR065"
+		(property "Reference" "#PWR047"
 			(at 109.22 77.47 0)
 			(effects
@@
 			(project "nuku-carrier-template-basic"
 				(path "/15e0a42f-48e0-4a5d-9b6b-7d249ffc02ad/cb35697b-7148-4b12-9d2d-66ae29597163"
-					(reference "#PWR065")
+					(reference "#PWR047")
 					(unit 1)
 				)
@@
 		(on_board yes)
 		(dnp no)
-		(property "Reference" "U10"
+		(property "Reference" "U7"
 			(at 231.14 93.98 0)
 			(effects
@@
 			(project "nuku-carrier-template-basic"
 				(path "/15e0a42f-48e0-4a5d-9b6b-7d249ffc02ad/cb35697b-7148-4b12-9d2d-66ae29597163"
-					(reference "U10")
+					(reference "U7")
 					(unit 1)
 				)
@@
 		(on_board yes)
 		(dnp no)
-		(property "Reference" "#PWR072"
+		(property "Reference" "#PWR054"
 			(at 167.64 124.46 0)
 			(effects
@@
 			(project "nuku-carrier-template-basic"
 				(path "/15e0a42f-48e0-4a5d-9b6b-7d249ffc02ad/cb35697b-7148-4b12-9d2d-66ae29597163"
-					(reference "#PWR072")
+					(reference "#PWR054")
 					(unit 1)
 				)
@@
 		(on_board yes)
 		(dnp no)
-		(property "Reference" "U8"
+		(property "Reference" "U5"
 			(at 176.53 93.98 0)
 			(effects
@@
 			(project "nuku-carrier-template-basic"
 				(path "/15e0a42f-48e0-4a5d-9b6b-7d249ffc02ad/cb35697b-7148-4b12-9d2d-66ae29597163"
-					(reference "U8")
+					(reference "U5")
 					(unit 1)
 				)
@@
 		(on_board yes)
 		(dnp no)
-		(property "Reference" "#PWR073"
+		(property "Reference" "#PWR055"
 			(at 222.25 49.53 0)
 			(effects
@@
 			(project "nuku-carrier-template-basic"
 				(path "/15e0a42f-48e0-4a5d-9b6b-7d249ffc02ad/cb35697b-7148-4b12-9d2d-66ae29597163"
-					(reference "#PWR073")
+					(reference "#PWR055")
 					(unit 1)
 				)
@@
 		(on_board yes)
 		(dnp no)
-		(property "Reference" "#PWR067"
+		(property "Reference" "#PWR049"
 			(at 111.76 73.66 0)
 			(effects
@@
 			(project "nuku-carrier-template-basic"
 				(path "/15e0a42f-48e0-4a5d-9b6b-7d249ffc02ad/cb35697b-7148-4b12-9d2d-66ae29597163"
-					(reference "#PWR067")
+					(reference "#PWR049")
 					(unit 1)
 				)
@@
 		(on_board yes)
 		(dnp no)
-		(property "Reference" "#PWR068"
+		(property "Reference" "#PWR050"
 			(at 111.76 118.11 0)
 			(effects
@@
 			(project "nuku-carrier-template-basic"
 				(path "/15e0a42f-48e0-4a5d-9b6b-7d249ffc02ad/cb35697b-7148-4b12-9d2d-66ae29597163"
-					(reference "#PWR068")
+					(reference "#PWR050")
 					(unit 1)
 				)
@@
 		(on_board yes)
 		(dnp no)
-		(property "Reference" "#PWR070"
+		(property "Reference" "#PWR052"
 			(at 167.64 80.01 0)
 			(effects
@@
 			(project "nuku-carrier-template-basic"
 				(path "/15e0a42f-48e0-4a5d-9b6b-7d249ffc02ad/cb35697b-7148-4b12-9d2d-66ae29597163"
-					(reference "#PWR070")
+					(reference "#PWR052")
 					(unit 1)
 				)
@@
 		(on_board yes)
 		(dnp no)
-		(property "Reference" "R43"
+		(property "Reference" "R30"
 			(at 71.12 153.67 90)
 			(effects
@@
 			(project "nuku-carrier-template-basic"
 				(path "/15e0a42f-48e0-4a5d-9b6b-7d249ffc02ad/cb35697b-7148-4b12-9d2d-66ae29597163"
-					(reference "R43")
+					(reference "R30")
 					(unit 1)
 				)
@@
 		(dnp no)
 		(fields_autoplaced yes)
-		(property "Reference" "#PWR078"
+		(property "Reference" "#PWR041"
 			(at 66.04 147.32 0)
 			(effects
@@
 			(project "nuku-carrier-template-basic"
 				(path "/15e0a42f-48e0-4a5d-9b6b-7d249ffc02ad/cb35697b-7148-4b12-9d2d-66ae29597163"
-					(reference "#PWR078")
+					(reference "#PWR041")
 					(unit 1)
 				)
@@
 		(on_board yes)
 		(dnp no)
-		(property "Reference" "#PWR076"
+		(property "Reference" "#PWR058"
 			(at 222.25 124.46 0)
 			(effects
@@
 			(project "nuku-carrier-template-basic"
 				(path "/15e0a42f-48e0-4a5d-9b6b-7d249ffc02ad/cb35697b-7148-4b12-9d2d-66ae29597163"
-					(reference "#PWR076")
+					(reference "#PWR058")
 					(unit 1)
 				)
@@
 		(on_board yes)
 		(dnp no)
-		(property "Reference" "#PWR074"
+		(property "Reference" "#PWR056"
 			(at 222.25 80.01 0)
 			(effects
@@
 			(project "nuku-carrier-template-basic"
 				(path "/15e0a42f-48e0-4a5d-9b6b-7d249ffc02ad/cb35697b-7148-4b12-9d2d-66ae29597163"
-					(reference "#PWR074")
+					(reference "#PWR056")
 					(unit 1)
 				)
@@
 		(on_board yes)
 		(dnp no)
-		(property "Reference" "#PWR079"
+		(property "Reference" "#PWR042"
 			(at 66.04 171.45 0)
 			(effects
@@
 			(project "nuku-carrier-template-basic"
 				(path "/15e0a42f-48e0-4a5d-9b6b-7d249ffc02ad/cb35697b-7148-4b12-9d2d-66ae29597163"
-					(reference "#PWR079")
+					(reference "#PWR042")
 					(unit 1)
 				)
@@
 		(on_board yes)
 		(dnp no)
-		(property "Reference" "#PWR066"
+		(property "Reference" "#PWR048"
 			(at 109.22 121.92 0)
 			(effects
@@
 			(project "nuku-carrier-template-basic"
 				(path "/15e0a42f-48e0-4a5d-9b6b-7d249ffc02ad/cb35697b-7148-4b12-9d2d-66ae29597163"
-					(reference "#PWR066")
+					(reference "#PWR048")
 					(unit 1)
 				)
@@
 		(on_board yes)
 		(dnp no)
-		(property "Reference" "U9"
+		(property "Reference" "U6"
 			(at 231.14 49.53 0)
 			(effects
@@
 			(project "nuku-carrier-template-basic"
 				(path "/15e0a42f-48e0-4a5d-9b6b-7d249ffc02ad/cb35697b-7148-4b12-9d2d-66ae29597163"
-					(reference "U9")
+					(reference "U6")
 					(unit 1)
 				)
@@
 		(on_board yes)
 		(dnp no)
-		(property "Reference" "#PWR069"
+		(property "Reference" "#PWR051"
 			(at 167.64 49.53 0)
 			(effects
@@
 			(project "nuku-carrier-template-basic"
 				(path "/15e0a42f-48e0-4a5d-9b6b-7d249ffc02ad/cb35697b-7148-4b12-9d2d-66ae29597163"
-					(reference "#PWR069")
+					(reference "#PWR051")
 					(unit 1)
 				)
@@
 		(on_board yes)
 		(dnp no)
-		(property "Reference" "#PWR063"
+		(property "Reference" "#PWR045"
 			(at 93.98 77.47 0)
 			(effects
@@
 			(project "nuku-carrier-template-basic"
 				(path "/15e0a42f-48e0-4a5d-9b6b-7d249ffc02ad/cb35697b-7148-4b12-9d2d-66ae29597163"
-					(reference "#PWR063")
+					(reference "#PWR045")
 					(unit 1)
 				)
@@
 		(on_board yes)
 		(dnp no)
-		(property "Reference" "#PWR075"
+		(property "Reference" "#PWR057"
 			(at 222.25 93.98 0)
 			(effects
@@
 			(project "nuku-carrier-template-basic"
 				(path "/15e0a42f-48e0-4a5d-9b6b-7d249ffc02ad/cb35697b-7148-4b12-9d2d-66ae29597163"
-					(reference "#PWR075")
+					(reference "#PWR057")
 					(unit 1)
 				)
@@
 		(on_board yes)
 		(dnp no)
-		(property "Reference" "U7"
+		(property "Reference" "U4"
 			(at 176.53 49.53 0)
 			(effects
@@
 			(project "nuku-carrier-template-basic"
 				(path "/15e0a42f-48e0-4a5d-9b6b-7d249ffc02ad/cb35697b-7148-4b12-9d2d-66ae29597163"
-					(reference "U7")
+					(reference "U4")
 					(unit 1)
 				)
@@
 		(dnp no)
 		(fields_autoplaced yes)
-		(property "Reference" "R42"
+		(property "Reference" "R29"
 			(at 68.58 158.7499 0)
 			(effects
@@
 			(project "nuku-carrier-template-basic"
 				(path "/15e0a42f-48e0-4a5d-9b6b-7d249ffc02ad/cb35697b-7148-4b12-9d2d-66ae29597163"
-					(reference "R42")
+					(reference "R29")
 					(unit 1)
 				)
