File: prj/nuku-carrier-template-bridgeless/nuku-carrier-template-bridgeless.kicad_pcb (KiCad board)
At the start: 4 copper layers, 90 x 40 mm, 57 parts, among them J1 DF40C-90DS-0.4V, J2 DF40C-90DS-0.4V, J3 DF40C-90DS-0.4V, J4 DF40C-90DS-0.4V, J5 USB_C_Receptacle_USB2.0_16P, J6 TC2050, J7 PMOD_A, J8 PMOD_B, SW1 PROG, SW2 RESET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

Commit message: Minor tweaks
Routing:
- net /core-south-0/CONFIG_DONE: track 38.0 -> 38.6 mm
Changed lines of the file:
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@@
+	)
+	(segment
+		(start 115.7 111.2)
+		(end 114.7 110.2)
+		(width 0.15)
+		(layer "F.Cu")
+		(net 24)
+	)
+	(segment
+		(start 119.9 115)
+		(end 119.3 114.4)
+		(width 0.15)
+		(layer "F.Cu")
+		(net 24)
+	)
+	(segment
+		(start 149.3 119.46)
+		(end 149.3 116.540041)
+		(width 0.15)
+		(layer "F.Cu")
+		(net 24)
+	)
+	(segment
+		(start 118.5 111.2)
+		(end 115.7 111.2)
+		(width 0.15)
+		(layer "F.Cu")
+		(net 24)
+	)
+	(segment
+		(start 114.7 100)
+		(end 112.7 98)
+		(width 0.15)
+		(layer "F.Cu")
+		(net 24)
+	)
+	(segment
+		(start 123.5 115)
+		(end 119.9 115)
+		(width 0.15)
+		(layer "F.Cu")
+		(net 24)
+	)
+	(segment
+		(start 111.9 95)
+		(end 109.81 95)
+		(width 0.15)
+		(layer "F.Cu")
+		(net 24)
+	)
+	(segment
+		(start 119.3 112)
+		(end 118.5 111.2)
+		(width 0.15)
+		(layer "F.Cu")
+		(net 24)
+	)
+	(segment
+		(start 114.7 110.2)
+		(end 114.7 100)
+		(width 0.15)
+		(layer "F.Cu")
+		(net 24)
+	)
+	(segment
+		(start 149.3 116.540041)
+		(end 148.359959 115.6)
+		(width 0.15)
+		(layer "F.Cu")
+		(net 24)
+	)
+	(segment
+		(start 148.359959 115.6)
+		(end 124.1 115.6)
+		(width 0.15)
+		(layer "F.Cu")
+		(net 24)
 	)
 	(segment
@@
 	)
 	(segment
-		(start 119.3 112)
-		(end 118.5 111.2)
-		(width 0.15)
-		(layer "F.Cu")
-		(net 24)
-	)
-	(segment
-		(start 115.7 111.2)
-		(end 114.7 110.2)
-		(width 0.15)
-		(layer "F.Cu")
-		(net 24)
-	)
-	(segment
-		(start 114.7 100)
-		(end 112.7 98)
-		(width 0.15)
-		(layer "F.Cu")
-		(net 24)
-	)
-	(segment
-		(start 118.5 111.2)
-		(end 115.7 111.2)
-		(width 0.15)
-		(layer "F.Cu")
-		(net 24)
-	)
-	(segment
-		(start 123.5 115)
-		(end 119.9 115)
+		(start 124.1 115.6)
+		(end 123.5 115)
 		(width 0.15)
 		(layer "F.Cu")
@@
 	)
 	(segment
-		(start 124.1 115.6)
-		(end 123.5 115)
-		(width 0.15)
-		(layer "F.Cu")
-		(net 24)
-	)
-	(segment
-		(start 149.3 119.46)
-		(end 149.3 117)
-		(width 0.15)
-		(layer "F.Cu")
-		(net 24)
-	)
-	(segment
-		(start 147.9 115.6)
-		(end 124.1 115.6)
-		(width 0.15)
-		(layer "F.Cu")
-		(net 24)
-	)
-	(segment
-		(start 111.9 95)
-		(end 109.81 95)
-		(width 0.15)
-		(layer "F.Cu")
-		(net 24)
-	)
-	(segment
-		(start 149.3 117)
-		(end 147.9 115.6)
-		(width 0.15)
-		(layer "F.Cu")
-		(net 24)
-	)
-	(segment
 		(start 109.81 93.8)
 		(end 109.81 95)
@@
 	)
 	(segment
-		(start 119.9 115)
-		(end 119.3 114.4)
-		(width 0.15)
-		(layer "F.Cu")
-		(net 24)
-	)
-	(segment
-		(start 114.7 110.2)
-		(end 114.7 100)
-		(width 0.15)
-		(layer "F.Cu")
-		(net 24)
-	)
-	(segment
 		(start 112.7 95.8)
 		(end 111.9 95)
@@
 	)
 	(segment
+		(start 115.9 116.6)
+		(end 115.9 118.89)
+		(width 0.15)
+		(layer "F.Cu")
+		(net 30)
+	)
+	(segment
+		(start 117.1 115.4)
+		(end 115.9 116.6)
+		(width 0.15)
+		(layer "F.Cu")
+		(net 30)
+	)
+	(segment
 		(start 148.5 116.8)
 		(end 147.7 116)
@@
 	)
 	(segment
-		(start 118.1 115.4)
-		(end 115.9 117.6)
-		(width 0.15)
-		(layer "F.Cu")
-		(net 30)
-	)
-	(segment
 		(start 123.3 115.4)
-		(end 118.1 115.4)
+		(end 117.1 115.4)
 		(width 0.15)
 		(layer "F.Cu")
@@
 	)
 	(segment
+		(start 147.7 116)
+		(end 123.9 116)
+		(width 0.15)
+		(layer "F.Cu")
+		(net 30)
+	)
+	(segment
 		(start 123.9 116)
 		(end 123.3 115.4)
-		(width 0.15)
-		(layer "F.Cu")
-		(net 30)
-	)
-	(segment
-		(start 115.9 117.6)
-		(end 115.9 118.89)
-		(width 0.15)
-		(layer "F.Cu")
-		(net 30)
-	)
-	(segment
-		(start 147.7 116)
-		(end 123.9 116)
 		(width 0.15)
 		(layer "F.Cu")
@@
 	)
 	(segment
+		(start 121.7 98.8)
+		(end 127.5 98.8)
+		(width 0.15)
+		(layer "F.Cu")
+		(net 189)
+	)
+	(segment
+		(start 148.3 92.6)
+		(end 149.7 94)
+		(width 0.15)
+		(layer "F.Cu")
+		(net 189)
+	)
+	(segment
+		(start 130.1 92.6)
+		(end 148.3 92.6)
+		(width 0.15)
+		(layer "F.Cu")
+		(net 189)
+	)
+	(segment
+		(start 121.665 96.435)
+		(end 121.3 96.8)
+		(width 0.15)
+		(layer "F.Cu")
+		(net 189)
+	)
+	(segment
+		(start 149.7 94)
+		(end 149.7 119.46)
+		(width 0.15)
+		(layer "F.Cu")
+		(net 189)
+	)
+	(segment
+		(start 127.5 98.8)
+		(end 128.7 97.6)
+		(width 0.15)
+		(layer "F.Cu")
+		(net 189)
+	)
+	(segment
+		(start 128.7 94)
+		(end 130.1 92.6)
+		(width 0.15)
+		(layer "F.Cu")
+		(net 189)
+	)
+	(segment
 		(start 121.3 98.4)
 		(end 121.7 98.8)
@@
 	)
 	(segment
-		(start 149.7 94.8)
-		(end 149.7 119.46)
-		(width 0.15)
-		(layer "F.Cu")
-		(net 189)
-	)
-	(segment
-		(start 121.7 98.8)
-		(end 127.5 98.8)
-		(width 0.15)
-		(layer "F.Cu")
-		(net 189)
-	)
-	(segment
-		(start 130.1 92.6)
-		(end 147.5 92.6)
-		(width 0.15)
-		(layer "F.Cu")
-		(net 189)
-	)
-	(segment
 		(start 122.8875 96.435)
 		(end 121.665 96.435)
@@
 	)
 	(segment
-		(start 147.5 92.6)
-		(end 149.7 94.8)
-		(width 0.15)
-		(layer "F.Cu")
-		(net 189)
-	)
-	(segment
-		(start 127.5 98.8)
-		(end 128.7 97.6)
-		(width 0.15)
-		(layer "F.Cu")
-		(net 189)
-	)
-	(segment
-		(start 121.665 96.435)
-		(end 121.3 96.8)
-		(width 0.15)
-		(layer "F.Cu")
-		(net 189)
-	)
-	(segment
-		(start 128.7 94)
-		(end 130.1 92.6)
+		(start 128.7 97.6)
+		(end 128.7 94)
 		(width 0.15)
 		(layer "F.Cu")
@@
 		(width 0.15)
 		(layer "F.Cu")
-		(net 189)
-	)
-	(segment
-		(start 128.7 97.6)
-		(end 128.7 94)
-		(width 0.15)
-		(layer "F.Cu")
