File: prj/nuku-carrier-template-bridgeless/nuku-carrier-template-bridgeless.kicad_pcb (KiCad board)
At the start: 4 copper layers, 90 x 40 mm, 57 parts, among them J1 DF40C-90DS-0.4V, J2 DF40C-90DS-0.4V, J3 DF40C-90DS-0.4V, J4 DF40C-90DS-0.4V, J5 USB_C_Receptacle_USB2.0_16P, J6 TC2050, J7 PMOD_A, J8 PMOD_B, SW1 PROG, SW2 RESET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

Commit message: Finish boards - prod ready
Routing:
- added copper zone on In2.Cu, net GND
- removed copper zone on In2.Cu, net (none)
Other:
- board text added: "90.0000 mm x 40.0000 mm"
- board text removed: "100.0000 mm x 60.0000 mm"
