File: prj/nuku-carrier-template-bridgeless/_autosave-nuku-carrier-template-bridgeless.kicad_pcb (KiCad board)
At the start: 4 copper layers, 90 x 40 mm, 57 parts, among them J1 DF40C-90DS-0.4V, J2 DF40C-90DS-0.4V, J3 DF40C-90DS-0.4V, J4 DF40C-90DS-0.4V, J5 USB_C_Receptacle_USB2.0_16P, J6 TC2050, J7 PMOD_A, J8 PMOD_B, SW1 PROG, SW2 RESET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

Commit message: Tweaks
Changed lines of the file:
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@@
-	)
-	(segment
-		(start 115.7 111.2)
-		(end 114.7 110.2)
-		(width 0.15)
-		(layer "F.Cu")
-		(net 24)
-	)
-	(segment
-		(start 119.9 115)
-		(end 119.3 114.4)
-		(width 0.15)
-		(layer "F.Cu")
-		(net 24)
-	)
-	(segment
-		(start 149.3 119.46)
-		(end 149.3 116.540041)
-		(width 0.15)
-		(layer "F.Cu")
-		(net 24)
-	)
-	(segment
-		(start 118.5 111.2)
-		(end 115.7 111.2)
-		(width 0.15)
-		(layer "F.Cu")
-		(net 24)
 	)
 	(segment
@@
 	)
 	(segment
-		(start 111.9 95)
-		(end 109.81 95)
+		(start 115.7 111.2)
+		(end 114.7 110.2)
 		(width 0.15)
 		(layer "F.Cu")
@@
 	)
 	(segment
-		(start 119.3 112)
-		(end 118.5 111.2)
+		(start 112.7 98)
+		(end 112.7 96.4)
+		(width 0.15)
+		(layer "F.Cu")
+		(net 24)
+	)
+	(segment
+		(start 149.3 116.540041)
+		(end 148.359959 115.6)
+		(width 0.15)
+		(layer "F.Cu")
+		(net 24)
+	)
+	(segment
+		(start 124.1 115.6)
+		(end 123.5 115)
+		(width 0.15)
+		(layer "F.Cu")
+		(net 24)
+	)
+	(segment
+		(start 119.3 114.4)
+		(end 119.3 111.8)
+		(width 0.15)
+		(layer "F.Cu")
+		(net 24)
+	)
+	(segment
+		(start 119.3 111.8)
+		(end 118.7 111.2)
+		(width 0.15)
+		(layer "F.Cu")
+		(net 24)
+	)
+	(segment
+		(start 118.7 111.2)
+		(end 115.7 111.2)
+		(width 0.15)
+		(layer "F.Cu")
+		(net 24)
+	)
+	(segment
+		(start 149.3 119.46)
+		(end 149.3 116.540041)
+		(width 0.15)
+		(layer "F.Cu")
+		(net 24)
+	)
+	(segment
+		(start 148.359959 115.6)
+		(end 124.1 115.6)
+		(width 0.15)
+		(layer "F.Cu")
+		(net 24)
+	)
+	(segment
+		(start 112.7 96.4)
+		(end 111.3 95)
 		(width 0.15)
 		(layer "F.Cu")
@@
 	)
 	(segment
-		(start 149.3 116.540041)
-		(end 148.359959 115.6)
-		(width 0.15)
-		(layer "F.Cu")
-		(net 24)
-	)
-	(segment
-		(start 148.359959 115.6)
-		(end 124.1 115.6)
-		(width 0.15)
-		(layer "F.Cu")
-		(net 24)
-	)
-	(segment
-		(start 119.3 114.4)
-		(end 119.3 112)
-		(width 0.15)
-		(layer "F.Cu")
-		(net 24)
-	)
-	(segment
-		(start 124.1 115.6)
-		(end 123.5 115)
-		(width 0.15)
-		(layer "F.Cu")
-		(net 24)
-	)
-	(segment
-		(start 112.7 98)
-		(end 112.7 95.8)
+		(start 119.9 115)
+		(end 119.3 114.4)
 		(width 0.15)
 		(layer "F.Cu")
@@
 	)
 	(segment
-		(start 112.7 95.8)
-		(end 111.9 95)
+		(start 111.3 95)
+		(end 109.81 95)
 		(width 0.15)
 		(layer "F.Cu")
