File: prj/nuku-carrier-template-bridgeless/power.kicad_sch (KiCad schematic)
At the start: 17 parts, among them J5 USB_C_Receptacle_USB2.0_16P, U1 AP61302

Commit message: Finish boards - prod ready
Parts:
- R23: now not fitted; now left out of the parts list
Changed lines of the file:
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@@
 		(unit 1)
 		(exclude_from_sim no)
-		(in_bom yes)
+		(in_bom no)
 		(on_board yes)
-		(dnp no)
+		(dnp yes)
 		(property "Reference" "R23"
 			(at 140.97 92.7099 0)
